Commit message: Add fan management.
Close #7 .

File: reachy_description/ros2_control/arm.ros2_control.xacro (robot description, xacro)
@@ -24,9 +24,27 @@
       <xacro:position_joint_control name="${name}_wrist_roll"/>
       <xacro:position_joint_control name="${name}_gripper"/>
-      <sensor name="${name}_gripper_force_sensor">
+      <sensor name="${name}_force_gripper">
         <state_interface name="force">
           <param name="initial_value">0.0</param>
         </state_interface>
-    </sensor>
+      </sensor>
+      <joint name="${name}_shoulder_fan">
+        <state_interface name="state">
+          <param name="initial_value">0.0</param>
+        </state_interface>
+        <command_interface name="state"/>
+      </joint>
+      <joint name="${name}_elbow_fan">
+        <state_interface name="state">
+          <param name="initial_value">0.0</param>
+        </state_interface>
+        <command_interface name="state"/>
+      </joint>
+      <joint name="${name}_wrist_fan">
+        <state_interface name="state">
+          <param name="initial_value">0.0</param>
+        </state_interface>
+        <command_interface name="state"/>
+      </joint>
     </ros2_control>
   </xacro:macro>

File: reachy_description/ros2_control/head.ros2_control.xacro (robot description, xacro)
@@ -19,4 +19,10 @@
       <xacro:position_joint_control name="neck_pitch"/>
       <xacro:position_joint_control name="neck_yaw"/>
+      <joint name="neck_fan">
+        <state_interface name="state">
+          <param name="initial_value">0.0</param>
+        </state_interface>
+        <command_interface name="state"/>
+      </joint>
     </ros2_control>
     <ros2_control name="antennas" type="system">
@@ -35,4 +41,16 @@
       <xacro:position_joint_control name="l_antenna"/>
       <xacro:position_joint_control name="r_antenna"/>
+      <joint name="l_antenna_fan">
+        <state_interface name="state">
+          <param name="initial_value">0.0</param>
+        </state_interface>
+        <command_interface name="state"/>
+      </joint>
+      <joint name="r_antenna_fan">
+        <state_interface name="state">
+          <param name="initial_value">0.0</param>
+        </state_interface>
+        <command_interface name="state"/>
+      </joint>
     </ros2_control>
   </xacro:macro>

Commit message: Use params for arm.

File: reachy_description/ros2_control/arm.ros2_control.xacro (robot description, xacro)
@@ -1,5 +1,5 @@
 <?xml version="1.0" ?>
 <robot xmlns:xacro="http://www.ros.org/wiki/xacro">
-  <xacro:macro name="arm_control" params="name">
+  <xacro:macro name="arm_control" params="name serial_port mx_ids offsets is_direct reductions force_sensor_id fan_id">
     <xacro:include filename="$(find reachy_description)/ros2_control/joint.ros2_control.xacro"/>
     <ros2_control name="${name}_arm" type="system">
@@ -7,11 +7,11 @@
         <xacro:unless value="$(arg use_fake_hardware)">
           <plugin>arm_system_hwi/ArmSystem</plugin>
-          <param name="serial_port">/dev/ttyACM0</param>
-          <param name="mx_ids">10, 11, 12, 13, 14, 15, 16, 17</param>
-          <param name="offsets">1.57, 1.57, 0.0, 0.0, 0.0, 0.0, 0.0, 0.0</param>
-          <param name="is_direct">0.0, 0.0, 0.0, 0.0, 0.0, 0.0, 0.0, 1.0</param>
-          <param name="reductions">1.0, 1.0, 1.0, 1.0, 1.0, 1.0, 1.0, -2.0</param>
-          <param name="force_sensor_id">40</param>
-          <param name="fan_id">41</param>
+          <param name="serial_port">${serial_port}</param>
+          <param name="mx_ids">${mx_ids}</param>
+          <param name="offsets">${offsets}</param>
+          <param name="is_direct">${is_direct}</param>
+          <param name="reductions">${reductions}</param>
+          <param name="force_sensor_id">${force_sensor_id}</param>
+          <param name="fan_id">${fan_id}</param>
         </xacro:unless>
         <xacro:if value="$(arg use_fake_hardware)">

File: reachy_description/urdf/arm.urdf.xacro (robot description, xacro)
@@ -1,5 +1,5 @@
 <?xml version="1.0"?>
 <robot xmlns:xacro="http://www.ros.org/wiki/xacro">
-<xacro:macro name="arm" params="prefix parent side damping friction">
+<xacro:macro name="arm" params="prefix parent side damping friction serial_port mx_ids offsets is_direct reductions force_sensor_id fan_id">
   <xacro:include filename="$(find reachy_description)/ros2_control/arm.ros2_control.xacro"/>
   <xacro:if value="${side == 'left'}">
@@ -238,5 +238,14 @@
       <dynamics damping="${damping}" friction="${friction}"/>
   </joint>
-  <xacro:arm_control name="${prefix}"/>
+  <xacro:arm_control
+    name="${prefix}"
+    serial_port="${serial_port}"
+    mx_ids="${mx_ids}"
+    offsets="${offsets}"
+    is_direct="${is_direct}"
+    reductions="${reductions}"
+    force_sensor_id="${force_sensor_id}"
+    fan_id="${fan_id}"
+  />
 </xacro:macro>
 </robot>

File: reachy_description/urdf/reachy.urdf.xacro (robot description, xacro)
@@ -41,4 +41,11 @@
     prefix="r" parent="torso" side="right"
     damping="${damping}" friction="${friction}"
+    serial_port="/dev/usb2ax_right_arm"
+    mx_ids="10, 11, 12, 13, 14, 15, 16, 17"
+    offsets="1.57, 1.57, 0.0, 0.0, 0.0, 0.0, 0.0, 0.0"
+    is_direct="0.0, 0.0, 0.0, 0.0, 0.0, 0.0, 0.0, 1.0"
+    reductions="1.0, 1.0, 1.0, 1.0, 1.0, 1.0, 1.0, -2.0"
+    force_sensor_id="40"
+    fan_id="41"
   />
   <!-- LEFT ARM-->
@@ -46,9 +53,16 @@
     prefix="l" parent="torso" side="left"
     damping="${damping}" friction="${friction}"
+    serial_port="/dev/usb2ax_left_arm"
+    mx_ids="20, 21, 22, 23, 24, 25, 26, 27"
+    offsets="1.57, -1.57, 0.0, 0.0, 0.0, 0.0, 0.0, 0.0"
+    is_direct="1.0, 0.0, 0.0, 0.0, 0.0, 0.0, 0.0, 1.0"
+    reductions="1.0, 1.0, 1.0, 1.0, 1.0, 1.0, 1.0, -2.0"
+    force_sensor_id="50"
+    fan_id="51"
   />
   <!-- HEAD-->
-  <xacro:head
+  <!-- <xacro:head
     parent="torso"
     damping="${damping}" friction="${friction}"
-  />
+  /> -->
 </robot>
