Commit message: simple test

File: reachy_description/ros2_control/head.ros2_control.xacro (robot description, xacro)
@@ -1,70 +1,71 @@
 <?xml version="1.0" ?>
 <robot xmlns:xacro="http://www.ros.org/wiki/xacro">
-  <xacro:macro name="head_control">
-    <xacro:include filename="$(find reachy_description)/ros2_control/joint.ros2_control.xacro"/>
-    <ros2_control name="head" type="system">
-      <hardware>
-        <xacro:unless value="$(arg use_fake_hardware)">
-          <!-- <plugin>head_system_hwi/HeadSystem</plugin> -->
-          <param name="serial_port">/dev/ttyACM0</param>
-          <param name="mx_ids"> 30, 31</param>
-          <param name="offsets">0.0, 0.0</param>
-          <param name="is_direct">0.0, 0.0</param>
-          <param name="reductions">0.0, 0.0</param>
-          <param name="fan_id">41</param>
-        </xacro:unless>
-        <xacro:if value="$(arg use_fake_hardware)">
-          <!-- Use gazebo as hardware simulation. -->
-          <xacro:if value="$(arg use_gazebo)">
-            <plugin>gazebo_ros2_control/GazeboSystem</plugin>
-          </xacro:if>
-          <!-- Use fake components. -->
-          <xacro:unless value="$(arg use_gazebo)">
-            <plugin>fake_components/GenericSystem</plugin>
-          </xacro:unless>
-        </xacro:if>
-      </hardware>
-      <xacro:position_joint_control name="neck_roll"/>
-      <xacro:position_joint_control name="neck_pitch"/>
-      <xacro:position_joint_control name="neck_yaw"/>
-      <joint name="neck_fan">
-        <state_interface name="state">
-          <param name="initial_value">0.0</param>
-        </state_interface>
-        <command_interface name="state"/>
-      </joint>
-    </ros2_control>
-    <ros2_control name="antennas" type="system">
-      <hardware>
-        <xacro:unless value="$(arg use_fake_hardware)">
-          <!-- <plugin>head_system_hwi/HeadSystem</plugin> -->
-          <plugin>fake_components/GenericSystem</plugin>
-        </xacro:unless>
-        <xacro:if value="$(arg use_fake_hardware)">
-          <!-- Use gazebo as hardware simulation. -->
-          <xacro:if value="$(arg use_gazebo)">
-            <plugin>gazebo_ros2_control/GazeboSystem</plugin>
-          </xacro:if>
-          <!-- Use fake components. -->
-          <xacro:unless value="$(arg use_gazebo)">
-            <plugin>fake_components/GenericSystem</plugin>
-          </xacro:unless>
-        </xacro:if>
-      </hardware>
-      <xacro:position_joint_control name="l_antenna"/>
-      <xacro:position_joint_control name="r_antenna"/>
-      <joint name="l_antenna_fan">
-        <state_interface name="state">
-          <param name="initial_value">0.0</param>
-        </state_interface>
-        <command_interface name="state"/>
-      </joint>
-      <joint name="r_antenna_fan">
-        <state_interface name="state">
-          <param name="initial_value">0.0</param>
-        </state_interface>
-        <command_interface name="state"/>
-      </joint>
-    </ros2_control>
-  </xacro:macro>
+    <xacro:macro name="head_control">
+        <xacro:include filename="$(find reachy_description)/ros2_control/joint.ros2_control.xacro"/>
+        <ros2_control name="head" type="system">
+            <hardware>
+                <xacro:unless value="$(arg use_fake_hardware)">
+                    <!--                    <plugin>head_system_hwi/HeadSystem</plugin>-->
+                    <plugin>fake_components/GenericSystem</plugin>
+                </xacro:unless>
+                <xacro:if value="$(arg use_fake_hardware)">
+                    <!-- Use gazebo as hardware simulation. -->
+                    <xacro:if value="$(arg use_gazebo)">
+                        <plugin>gazebo_ros2_control/GazeboSystem</plugin>
+                    </xacro:if>
+                    <!-- Use fake components. -->
+                    <xacro:unless value="$(arg use_gazebo)">
+                        <plugin>fake_components/GenericSystem</plugin>
+                    </xacro:unless>
+                </xacro:if>
+            </hardware>
+            <!--      <xacro:position_joint_control name="neck_roll"/>-->
+            <!--      <xacro:position_joint_control name="neck_pitch"/>-->
+            <!--      <xacro:position_joint_control name="neck_yaw"/>-->
+            <!--      <joint name="neck_fan">-->
+            <!--        <state_interface name="state">-->
+            <!--          <param name="initial_value">0.0</param>-->
+            <!--        </state_interface>-->
+            <!--        <command_interface name="state"/>-->
+            <!--      </joint>-->
+        </ros2_control>
+        <ros2_control name="antennas" type="system">
+            <hardware>
+                <xacro:unless value="$(arg use_fake_hardware)">
+                    <plugin>head_system_hwi/HeadSystem</plugin>
+                    <param name="serial_port">/dev/ttyACM0</param>
+                    <param name="mx_ids">30, 31</param>
+                    <param name="offsets">0.0, 0.0</param>
+                    <param name="is_direct">0.0, 0.0</param>
+                    <param name="reductions">0.0, 0.0</param>
+                    <param name="fan_id">41</param>
+                    <!--          <plugin>fake_components/GenericSystem</plugin>-->
+                </xacro:unless>
+                <xacro:if value="$(arg use_fake_hardware)">
+                    <!-- Use gazebo as hardware simulation. -->
+                    <xacro:if value="$(arg use_gazebo)">
+                        <plugin>gazebo_ros2_control/GazeboSystem</plugin>
+                    </xacro:if>
+                    <!-- Use fake components. -->
+                    <xacro:unless value="$(arg use_gazebo)">
+                        <plugin>fake_components/GenericSystem</plugin>
+                    </xacro:unless>
+                </xacro:if>
+            </hardware>
+            <xacro:position_joint_control name="l_antenna"/>
+            <xacro:position_joint_control name="r_antenna"/>
+<!--            <joint name="l_antenna_fan">-->
+<!--                <state_interface name="state">-->
+<!--                    <param name="initial_value">0.0</param>-->
+<!--                </state_interface>-->
+<!--                <command_interface name="state"/>-->
+<!--            </joint>-->
+<!--            <joint name="r_antenna_fan">-->
+<!--                <state_interface name="state">-->
+<!--                    <param name="initial_value">0.0</param>-->
+<!--                </state_interface>-->
+<!--                <command_interface name="state"/>-->
+<!--            </joint>-->
+        </ros2_control>
+    </xacro:macro>
 </robot>

Commit message: fan control seems ok through grpc

File: reachy_description/ros2_control/head.ros2_control.xacro (robot description, xacro)
@@ -39,5 +39,5 @@
                     <param name="is_direct">0.0, 0.0</param>
                     <param name="reductions">1.0, 1.0</param>
-                    <param name="fan_id">41</param>
+                    <param name="fan_id">40</param>
                     <!--          <plugin>fake_components/GenericSystem</plugin>-->
                 </xacro:unless>
@@ -55,16 +55,16 @@
             <xacro:position_joint_control name="l_antenna"/>
             <xacro:position_joint_control name="r_antenna"/>
-<!--            <joint name="l_antenna_fan">-->
-<!--                <state_interface name="state">-->
-<!--                    <param name="initial_value">0.0</param>-->
-<!--                </state_interface>-->
-<!--                <command_interface name="state"/>-->
-<!--            </joint>-->
-<!--            <joint name="r_antenna_fan">-->
-<!--                <state_interface name="state">-->
-<!--                    <param name="initial_value">0.0</param>-->
-<!--                </state_interface>-->
-<!--                <command_interface name="state"/>-->
-<!--            </joint>-->
+            <joint name="l_antenna_fan">
+                <state_interface name="state">
+                    <param name="initial_value">0.0</param>
+                </state_interface>
+                <command_interface name="state"/>
+            </joint>
+            <joint name="r_antenna_fan">
+                <state_interface name="state">
+                    <param name="initial_value">0.0</param>
+                </state_interface>
+                <command_interface name="state"/>
+            </joint>
         </ros2_control>
     </xacro:macro>

Commit message: Add fake orbita joints in head.
Also update ACM port for the head according to udev rules.

File: reachy_description/ros2_control/head.ros2_control.xacro (robot description, xacro)
@@ -20,13 +20,13 @@
                 </xacro:if>
             </hardware>
-            <!--      <xacro:position_joint_control name="neck_roll"/>-->
-            <!--      <xacro:position_joint_control name="neck_pitch"/>-->
-            <!--      <xacro:position_joint_control name="neck_yaw"/>-->
+                 <xacro:position_joint_control name="neck_roll"/>
+                 <xacro:position_joint_control name="neck_pitch"/>
+                 <xacro:position_joint_control name="neck_yaw"/>
             <!--      <joint name="neck_fan">-->
-            <!--        <state_interface name="state">-->
-            <!--          <param name="initial_value">0.0</param>-->
-            <!--        </state_interface>-->
-            <!--        <command_interface name="state"/>-->
-            <!--      </joint>-->
+                   <!-- <state_interface name="state">
+                     <param name="initial_value">0.0</param>
+                   </state_interface> -->
+                   <!-- <command_interface name="state"/> -->
+                 <!-- </joint> -->
         </ros2_control>
         <ros2_control name="antennas" type="system">
@@ -34,5 +34,5 @@
                 <xacro:unless value="$(arg use_fake_hardware)">
                     <plugin>head_system_hwi/HeadSystem</plugin>
-                    <param name="serial_port">/dev/ttyACM0</param>
+                    <param name="serial_port">/dev/usb2ax_head</param>
                     <param name="xl320_ids">30, 31</param>
                     <param name="offsets">0.0, 0.0</param>

Commit message: Remove neck fan.

File: reachy_description/ros2_control/head.ros2_control.xacro (robot description, xacro)
@@ -23,10 +23,4 @@
                  <xacro:position_joint_control name="neck_pitch"/>
                  <xacro:position_joint_control name="neck_yaw"/>
-            <!--      <joint name="neck_fan">-->
-                   <!-- <state_interface name="state">
-                     <param name="initial_value">0.0</param>
-                   </state_interface> -->
-                   <!-- <command_interface name="state"/> -->
-                 <!-- </joint> -->
         </ros2_control>
         <ros2_control name="antennas" type="system">

Commit message: Setup params for neck and head.

File: reachy_description/ros2_control/head.ros2_control.xacro (robot description, xacro)
@@ -1,5 +1,5 @@
 <?xml version="1.0" ?>
 <robot xmlns:xacro="http://www.ros.org/wiki/xacro">
-    <xacro:macro name="head_control">
+    <xacro:macro name="head_control" params="neck_orbita_serial_port neck_orbita_id neck_orbita_alpha neck_orbita_hardware_zero neck_orbita_encoder_resolution neck_orbita_reduction head_serial_port head_xl320_ids head_xl320_offsets head_xl320_is_direct head_xl320_reductions head_fan_id">
         <xacro:include filename="$(find reachy_description)/ros2_control/joint.ros2_control.xacro"/>
         <ros2_control name="head" type="system">
@@ -7,6 +7,10 @@
                 <xacro:unless value="$(arg use_fake_hardware)">
                     <plugin>neck_system_hwi/NeckSystem</plugin>
-                    <param name="serial_port">/dev/neck</param>
-                    <param name="offsets">0.0, 0.0, 0.0</param>
+                    <param name="serial_port">${neck_orbita_serial_port}</param>
+                    <param name="id">${neck_orbita_id}</param>
+                    <param name="alpha">${neck_orbita_alpha}</param>
+                    <param name="hardware_zero">${neck_orbita_hardware_zero}</param>
+                    <param name="encoder_resolution">${neck_orbita_encoder_resolution}</param>
+                    <param name="reduction">${neck_orbita_reduction}</param>
                 </xacro:unless>
                 <xacro:if value="$(arg use_fake_hardware)">
@@ -29,11 +33,10 @@
                 <xacro:unless value="$(arg use_fake_hardware)">
                     <plugin>head_system_hwi/HeadSystem</plugin>
-                    <param name="serial_port">/dev/usb2ax_head</param>
-                    <param name="xl320_ids">30, 31</param>
-                    <param name="offsets">0.0, 0.0</param>
-                    <param name="is_direct">0.0, 0.0</param>
-                    <param name="reductions">1.0, 1.0</param>
-                    <param name="fan_id">60</param>
-                    <!--          <plugin>fake_components/GenericSystem</plugin>-->
+                    <param name="serial_port">${head_serial_port}</param>
+                    <param name="xl320_ids">${head_xl320_ids}</param>
+                    <param name="offsets">${head_xl320_offsets}</param>
+                    <param name="is_direct">${head_xl320_is_direct}</param>
+                    <param name="reductions">${head_xl320_reductions}</param>
+                    <param name="fan_id">${head_fan_id}</param>
                 </xacro:unless>
                 <xacro:if value="$(arg use_fake_hardware)">

File: reachy_description/urdf/head.urdf.xacro (robot description, xacro)
@@ -4,5 +4,5 @@
   <xacro:property name="camera_link" value="0.05" /> <!-- Size of square 'camera' box -->
   <xacro:property name="camera_convergence" value="0.0" /> <!-- convergence angle (rad) of the cameras. 0=parallel-->
-  <xacro:macro name="head" params="parent damping friction">
+  <xacro:macro name="head" params="parent damping friction neck_orbita_serial_port neck_orbita_id neck_orbita_alpha neck_orbita_hardware_zero neck_orbita_encoder_resolution neck_orbita_reduction head_serial_port head_xl320_ids head_xl320_offsets head_xl320_is_direct head_xl320_reductions head_fan_id">
     <xacro:include filename="$(find reachy_description)/ros2_control/head.ros2_control.xacro"/>
     <joint name="neck_roll" type="revolute">
@@ -211,5 +211,18 @@
       <limit lower="-2.618" upper="2.618" effort="10." velocity="0.0"/>
     </joint>
-    <xacro:head_control/>
+    <xacro:head_control
+      neck_orbita_serial_port="${neck_orbita_serial_port}"
+      neck_orbita_id="${neck_orbita_id}"
+      neck_orbita_alpha="${neck_orbita_alpha}"
+      neck_orbita_hardware_zero="${neck_orbita_hardware_zero}"
+      neck_orbita_encoder_resolution="${neck_orbita_encoder_resolution}"
+      neck_orbita_reduction="${neck_orbita_reduction}"
+      head_serial_port="${head_serial_port}"
+      head_xl320_ids="${head_xl320_ids}"
+      head_xl320_offsets="${head_xl320_offsets}"
+      head_xl320_is_direct="${head_xl320_is_direct}"
+      head_xl320_reductions="${head_xl320_reductions}"
+      head_fan_id="${head_fan_id}"
+    />
     <!-- Cameras -->
     <xacro:if value="$(arg use_gazebo)">

File: reachy_description/urdf/reachy.urdf.xacro (robot description, xacro)
@@ -87,4 +87,16 @@
       parent="torso"
       damping="${damping}" friction="${friction}"
+      neck_orbita_serial_port="/dev/usb2orbita_neck"
+      neck_orbita_id="70"
+      neck_orbita_alpha="54.0"
+      neck_orbita_hardware_zero="0.0, 0.0, 0.0"
+      neck_orbita_encoder_resolution="4096"
+      neck_orbita_reduction="4.0"
+      head_serial_port="/dev/usb2ax_head"
+      head_xl320_ids="30, 31"
+      head_xl320_offsets="0.0, 0.0"
+      head_xl320_is_direct="0.0, 0.0"
+      head_xl320_reductions="1.0, 1.0"
+      head_fan_id="60"
     />
   </xacro:if>

Commit message: Remove unused encoder res.

File: reachy_description/ros2_control/head.ros2_control.xacro (robot description, xacro)
@@ -1,5 +1,5 @@
 <?xml version="1.0" ?>
 <robot xmlns:xacro="http://www.ros.org/wiki/xacro">
-    <xacro:macro name="head_control" params="neck_orbita_serial_port neck_orbita_id neck_orbita_alpha neck_orbita_hardware_zero neck_orbita_encoder_resolution neck_orbita_reduction head_serial_port head_xl320_ids head_xl320_offsets head_xl320_is_direct head_xl320_reductions head_fan_id">
+    <xacro:macro name="head_control" params="neck_orbita_serial_port neck_orbita_id neck_orbita_alpha neck_orbita_hardware_zero neck_orbita_reduction head_serial_port head_xl320_ids head_xl320_offsets head_xl320_is_direct head_xl320_reductions head_fan_id">
         <xacro:include filename="$(find reachy_description)/ros2_control/joint.ros2_control.xacro"/>
         <ros2_control name="head" type="system">
@@ -11,5 +11,4 @@
                     <param name="alpha">${neck_orbita_alpha}</param>
                     <param name="hardware_zero">${neck_orbita_hardware_zero}</param>
-                    <param name="encoder_resolution">${neck_orbita_encoder_resolution}</param>
                     <param name="reduction">${neck_orbita_reduction}</param>
                 </xacro:unless>

File: reachy_description/urdf/head.urdf.xacro (robot description, xacro)
@@ -4,5 +4,5 @@
   <xacro:property name="camera_link" value="0.05" /> <!-- Size of square 'camera' box -->
   <xacro:property name="camera_convergence" value="0.0" /> <!-- convergence angle (rad) of the cameras. 0=parallel-->
-  <xacro:macro name="head" params="parent damping friction neck_orbita_serial_port neck_orbita_id neck_orbita_alpha neck_orbita_hardware_zero neck_orbita_encoder_resolution neck_orbita_reduction head_serial_port head_xl320_ids head_xl320_offsets head_xl320_is_direct head_xl320_reductions head_fan_id">
+  <xacro:macro name="head" params="parent damping friction neck_orbita_serial_port neck_orbita_id neck_orbita_alpha neck_orbita_hardware_zero neck_orbita_reduction head_serial_port head_xl320_ids head_xl320_offsets head_xl320_is_direct head_xl320_reductions head_fan_id">
     <xacro:include filename="$(find reachy_description)/ros2_control/head.ros2_control.xacro"/>
     <joint name="neck_roll" type="revolute">
@@ -216,5 +216,4 @@
       neck_orbita_alpha="${neck_orbita_alpha}"
       neck_orbita_hardware_zero="${neck_orbita_hardware_zero}"
-      neck_orbita_encoder_resolution="${neck_orbita_encoder_resolution}"
       neck_orbita_reduction="${neck_orbita_reduction}"
       head_serial_port="${head_serial_port}"

File: reachy_description/urdf/reachy.urdf.xacro (robot description, xacro)
@@ -91,5 +91,4 @@
       neck_orbita_alpha="54.0"
       neck_orbita_hardware_zero="0.0, 0.0, 0.0"
-      neck_orbita_encoder_resolution="4096"
       neck_orbita_reduction="4.0"
       head_serial_port="/dev/usb2ax_head"
