Commit message: kinematics ok

File: reachy_description/urdf/head.urdf.xacro (robot description, xacro)
@@ -149,4 +149,14 @@
       </collision>
     </link>
+    <link name="head_tip" >
+    </link>
+    <joint name="head_tip_fixed" type="fixed">
+      <!-- between the cameras -->
+      <!-- <origin xyz="0.02 0 0.06105" rpy="0.0 0.0 0"/> -->
+      <!-- Rotation center -->
+      <origin xyz="0.0 0 0.0" rpy="0.0 0.0 0"/>
+      <parent link="head" />
+      <child link="head_tip" />
+    </joint>
     <link name="l_antenna_link">
       <inertial>

Commit message: head cartesian kinematics

File: reachy_description/urdf/head.urdf.xacro (robot description, xacro)
@@ -153,7 +153,7 @@
     <joint name="head_tip_fixed" type="fixed">
       <!-- between the cameras -->
-      <!-- <origin xyz="0.02 0 0.06105" rpy="0.0 0.0 0"/> -->
+      <origin xyz="0.02 0 0.06105" rpy="0.0 0.0 0"/>
       <!-- Rotation center -->
-      <origin xyz="0.0 0 0.0" rpy="0.0 0.0 0"/>
+      <!-- <origin xyz="0.0 0 0.0" rpy="0.0 0.0 0"/> -->
       <parent link="head" />
       <child link="head_tip" />

Commit message: Update head.urdf.xacro

File: reachy_description/urdf/head.urdf.xacro (robot description, xacro)
@@ -7,5 +7,5 @@
     <xacro:include filename="$(find reachy_description)/ros2_control/head.ros2_control.xacro"/>
     <joint name="neck_roll" type="revolute">
-      <origin xyz="0.015 0.0 0.095" rpy="0 0.174 0" />
+      <origin xyz="0.015 0.0 0.095" rpy="-0.15105105 0.08669986 -1.05356462"/>
       <parent link="${parent}"/>
       <child link="head_x"/>
@@ -52,5 +52,5 @@
     </link>
     <joint name="neck_fixed" type="fixed">
-      <origin xyz="0 0 0" rpy="0.0 0.0 0.0"/>
+      <origin xyz="0 0 0" rpy="0.0 0.0 1.047"/>
       <parent link="head_z" />
       <child link="head" />
