Commit message: Ros control (#2)
* Create reachy_bringup, reachy_sdk_server, pid_command_controller, arm_system_hwi,
* Setup ros2 control with controllers, config files,
* Setup grpc communication,
* Fix #6 #7 #8 #9.

File: reachy_description/urdf/arm.urdf.xacro (robot description, xacro)
@@ -1,5 +1,6 @@
 <?xml version="1.0"?>
 <robot xmlns:xacro="http://www.ros.org/wiki/xacro">
-<xacro:macro name="arm" params="prefix parent side damping friction">
+<xacro:macro name="arm" params="prefix parent side damping friction serial_port mx_ids offsets is_direct reductions force_sensor_id fan_id">
+  <xacro:include filename="$(find reachy_description)/ros2_control/arm.ros2_control.xacro"/>
   <xacro:if value="${side == 'left'}">
     <xacro:property name="reflect" value="-1"/>
@@ -237,4 +238,14 @@
       <dynamics damping="${damping}" friction="${friction}"/>
   </joint>
+  <xacro:arm_control
+    name="${prefix}"
+    serial_port="${serial_port}"
+    mx_ids="${mx_ids}"
+    offsets="${offsets}"
+    is_direct="${is_direct}"
+    reductions="${reductions}"
+    force_sensor_id="${force_sensor_id}"
+    fan_id="${fan_id}"
+  />
 </xacro:macro>
 </robot>

File: reachy_description/urdf/head.urdf.xacro (robot description, xacro)
@@ -2,4 +2,5 @@
 <robot xmlns:xacro="http://www.ros.org/wiki/xacro">
 <xacro:macro name="head" params="parent damping friction">
+  <xacro:include filename="$(find reachy_description)/ros2_control/head.ros2_control.xacro"/>
   <joint name="neck_roll" type="revolute">
       <origin xyz="0.015 0.0 0.095" rpy="0 0.174 0" />
@@ -164,4 +165,5 @@
     <limit lower="-2.618" upper="2.618" effort="10." velocity="0.0"/>
   </joint>
+  <xacro:head_control/>
 </xacro:macro>
 </robot>

File: reachy_description/urdf/reachy.urdf.xacro (robot description, xacro)
@@ -1,4 +1,6 @@
 <?xml version="1.0"?>
 <robot xmlns:xacro="http://www.ros.org/wiki/xacro" name="reachy_2023">
+  <xacro:arg name="use_fake_hardware" default="false"/>
+  <xacro:arg name="use_gazebo" default="false"/>
   <xacro:include filename="$(find reachy_description)/urdf/arm.urdf.xacro"/>
   <xacro:include filename="$(find reachy_description)/urdf/head.urdf.xacro"/>
@@ -39,4 +41,11 @@
     prefix="r" parent="torso" side="right"
     damping="${damping}" friction="${friction}"
+    serial_port="/dev/usb2ax_right_arm"
+    mx_ids="10, 11, 12, 13, 14, 15, 16, 17"
+    offsets="1.57, 1.57, 0.0, 0.0, 0.0, 0.0, 0.0, 0.0"
+    is_direct="0.0, 0.0, 0.0, 0.0, 0.0, 0.0, 0.0, 1.0"
+    reductions="1.0, 1.0, 1.0, 1.0, 1.0, 1.0, 1.0, -2.0"
+    force_sensor_id="40"
+    fan_id="41"
   />
   <!-- LEFT ARM-->
@@ -44,9 +53,16 @@
     prefix="l" parent="torso" side="left"
     damping="${damping}" friction="${friction}"
+    serial_port="/dev/usb2ax_left_arm"
+    mx_ids="20, 21, 22, 23, 24, 25, 26, 27"
+    offsets="1.57, -1.57, 0.0, 0.0, 0.0, 0.0, 0.0, 0.0"
+    is_direct="1.0, 0.0, 0.0, 0.0, 0.0, 0.0, 0.0, 1.0"
+    reductions="1.0, 1.0, 1.0, 1.0, 1.0, 1.0, 1.0, -2.0"
+    force_sensor_id="50"
+    fan_id="51"
   />
   <!-- HEAD-->
-  <xacro:head
+  <!-- <xacro:head
     parent="torso"
     damping="${damping}" friction="${friction}"
-  />
+  /> -->
 </robot>

Commit message: gazebo seems okish

File: reachy_description/urdf/arm.urdf.xacro (robot description, xacro)
@@ -20,5 +20,5 @@
           <origin xyz="0.0 ${0.04*reflect} 0.0" rpy="${1.57*reflect} 1.57 0.0"/>
           <geometry>
-              <mesh filename="package://reachy_description/meshes/shoulder.dae"/>
+              <mesh filename="file://$(find reachy_description)/meshes/shoulder.dae"/>
           </geometry>
       </visual>
@@ -47,5 +47,5 @@
           <origin xyz="0.0 0.0 0.0" rpy="0.0 0.0 0.0"/>
           <geometry>
-              <mesh filename="package://reachy_description/meshes/shoulder_x.dae"/>
+              <mesh filename="file://$(find reachy_description)/meshes/shoulder_x.dae"/>
           </geometry>
       </visual>
@@ -79,5 +79,5 @@
           <origin xyz="0.0 0.0 -0.0526" rpy="0.0 0.0 0.0"/>
           <geometry>
-              <mesh filename="package://reachy_description/meshes/upper_arm.dae"/>
+              <mesh filename="file://$(find reachy_description)/meshes/upper_arm.dae"/>
           </geometry>
       </visual>
@@ -106,5 +106,5 @@
           <origin xyz="0.0 0.0 0.0" rpy="0.0 0.0 0.0"/>
           <geometry>
-              <mesh filename="package://reachy_description/meshes/forearm.dae"/>
+              <mesh filename="file://$(find reachy_description)/meshes/forearm.dae"/>
           </geometry>
       </visual>
@@ -133,5 +133,5 @@
           <origin xyz="0.0 0.0 -0.100" rpy="0.0 0.0 0.0"/>
           <geometry>
-              <mesh filename="package://reachy_description/meshes/wrist.dae"/>
+              <mesh filename="file://$(find reachy_description)/meshes/wrist.dae"/>
           </geometry>
       </visual>
@@ -160,5 +160,5 @@
           <origin xyz="0.0 0.0 0.0" rpy="0.0 0.0 0.0"/>
           <geometry>
-              <mesh filename="package://reachy_description/meshes/wrist2hand.dae"/>
+              <mesh filename="file://$(find reachy_description)/meshes/wrist2hand.dae"/>
           </geometry>
       </visual>
@@ -187,5 +187,5 @@
           <origin xyz="0.0 0.0 0.0" rpy="0.0 1.57 0.0"/>
           <geometry>
-              <mesh filename="package://reachy_description/meshes/${prefix}_gripper_thumb.dae"/>
+              <mesh filename="file://$(find reachy_description)/meshes/${prefix}_gripper_thumb.dae"/>
           </geometry>
       </visual>
@@ -214,5 +214,5 @@
           <origin xyz="0.0 0.0 0.0" rpy="0.0 1.57 0.0"/>
           <geometry>
-              <mesh filename="package://reachy_description/meshes/${prefix}_gripper_finger.dae"/>
+              <mesh filename="file://$(find reachy_description)/meshes/${prefix}_gripper_finger.dae"/>
           </geometry>
       </visual>
@@ -224,5 +224,11 @@
       </collision>
   </link>
-  <link name="${prefix}_arm_tip"/>
+  <link name="${prefix}_arm_tip">
+    <inertial>
+          <origin xyz="0.0 0.0 0.0" rpy="0.0 0.0 0.0"/>
+          <mass value="0.001"/>
+          <inertia ixx="1.0e-6" ixy="1.0e-8" ixz="1.0e-8" iyy="1.0e-6" iyz="1.0e-8" izz="1.0e-6"/>
+    </inertial>
+    </link>
   <joint name="${prefix}_arm_tip" type="fixed">
       <origin xyz="0 -0.012 -0.085" rpy="0 0 0" />

File: reachy_description/urdf/head.urdf.xacro (robot description, xacro)
@@ -11,5 +11,11 @@
     <dynamics damping="${damping}" friction="${friction}"/>
   </joint>
-  <link name="head_x" />
+  <link name="head_x">
+    <inertial>
+          <origin xyz="0.0 0.0 0.0" rpy="0.0 0.0 0.0"/>
+          <mass value="0.001"/>
+          <inertia ixx="1.0e-6" ixy="1.0e-8" ixz="1.0e-8" iyy="1.0e-6" iyz="1.0e-8" izz="1.0e-6"/>
+    </inertial>
+    </link>
   <joint name="neck_pitch" type="revolute">
       <origin xyz="0 0 0" rpy="0.0 0.0 0.0"/>
@@ -20,5 +26,11 @@
     <dynamics damping="${damping}" friction="${friction}"/>
   </joint>
-  <link name="head_y" />
+  <link name="head_y" >
+    <inertial>
+          <origin xyz="0.0 0.0 0.0" rpy="0.0 0.0 0.0"/>
+          <mass value="0.001"/>
+          <inertia ixx="1.0e-6" ixy="1.0e-8" ixz="1.0e-8" iyy="1.0e-6" iyz="1.0e-8" izz="1.0e-6"/>
+    </inertial>
+    </link>
   <joint name="neck_yaw" type="revolute">
       <origin xyz="0 0 0" rpy="0.0 0.0 0.0"/>
@@ -29,5 +41,11 @@
     <dynamics damping="${damping}" friction="${friction}"/>
   </joint>
-  <link name="head_z" />
+  <link name="head_z">
+    <inertial>
+          <origin xyz="0.0 0.0 0.0" rpy="0.0 0.0 0.0"/>
+          <mass value="0.001"/>
+          <inertia ixx="1.0e-6" ixy="1.0e-8" ixz="1.0e-8" iyy="1.0e-6" iyz="1.0e-8" izz="1.0e-6"/>
+    </inertial>
+  </link>
   <joint name="neck_fixed" type="fixed">
       <origin xyz="0 0 0" rpy="0.0 0.0 0.0"/>
@@ -42,8 +60,13 @@
   </joint>
   <link name="top_neck_arm">
+    <inertial>
+          <origin xyz="0.0 0.0 0.0" rpy="0.0 0.0 0.0"/>
+          <mass value="0.001"/>
+          <inertia ixx="1.0e-6" ixy="1.0e-8" ixz="1.0e-8" iyy="1.0e-6" iyz="1.0e-8" izz="1.0e-6"/>
+    </inertial>
       <visual name="">
           <origin xyz="0.0 0.0 0.0" rpy="0.0 0.0 0.5236"/>
           <geometry>
-              <mesh filename="package://reachy_description/meshes/orbita_arm.dae"/>
+              <mesh filename="file://$(find reachy_description)/meshes/orbita_arm.dae"/>
           </geometry>
       </visual>
@@ -61,8 +84,13 @@
   </joint>
   <link name="middle_neck_arm">
+    <inertial>
+          <origin xyz="0.0 0.0 0.0" rpy="0.0 0.0 0.0"/>
+          <mass value="0.001"/>
+          <inertia ixx="1.0e-6" ixy="1.0e-8" ixz="1.0e-8" iyy="1.0e-6" iyz="1.0e-8" izz="1.0e-6"/>
+    </inertial>
       <visual name="">
           <origin xyz="0.0 0.0 0.0" rpy="0.0 0.0 2.618"/>
           <geometry>
-              <mesh filename="package://reachy_description/meshes/orbita_arm.dae"/>
+              <mesh filename="file://$(find reachy_description)/meshes/orbita_arm.dae"/>
           </geometry>
       </visual>
@@ -80,8 +108,13 @@
   </joint>
   <link name="bottom_neck_arm">
+    <inertial>
+          <origin xyz="0.0 0.0 0.0" rpy="0.0 0.0 0.0"/>
+          <mass value="0.001"/>
+          <inertia ixx="1.0e-6" ixy="1.0e-8" ixz="1.0e-8" iyy="1.0e-6" iyz="1.0e-8" izz="1.0e-6"/>
+    </inertial>
       <visual name="">
           <origin xyz="0.0 0.0 0.0" rpy="0.0 0.0 -1.57"/>
           <geometry>
-              <mesh filename="package://reachy_description/meshes/orbita_arm.dae"/>
+              <mesh filename="file://$(find reachy_description)/meshes/orbita_arm.dae"/>
           </geometry>
       </visual>
@@ -103,5 +136,5 @@
           <origin xyz="0.0 0.0 0.0" rpy="0.0 0.0 0.0"/>
           <geometry>
-              <mesh filename="package://reachy_description/meshes/head.dae"/>
+              <mesh filename="file://$(find reachy_description)/meshes/head.dae"/>
           </geometry>
       </visual>
@@ -122,5 +155,5 @@
           <origin xyz="0.0 0.0 0.0" rpy="0.0 0.0 0.0"/>
           <geometry>
-              <mesh filename="package://reachy_description/meshes/antenna.dae"/>
+              <mesh filename="file://$(find reachy_description)/meshes/antenna.dae"/>
           </geometry>
       </visual>
@@ -148,5 +181,5 @@
           <origin xyz="0.0 0.0 0.0" rpy="0.0 0.0 0.0"/>
           <geometry>
-              <mesh filename="package://reachy_description/meshes/antenna.dae"/>
+              <mesh filename="file://$(find reachy_description)/meshes/antenna.dae"/>
           </geometry>
       </visual>

File: reachy_description/urdf/reachy.urdf.xacro (robot description, xacro)
@@ -20,5 +20,5 @@
           <origin xyz="0.0 0.0 0.0" rpy="0.0 0.0 0.0"/>
           <geometry>
-              <mesh filename="package://reachy_description/meshes/torso.dae"/>
+              <mesh filename="file://$(find reachy_description)/meshes/torso.dae"/>
           </geometry>
       </visual>
@@ -31,5 +31,5 @@
   </link>
   <gazebo reference="torso">
-    <material>Gazebo/Black</material>
+    <material>Gazebo/White</material>
     <static>true</static>
   </gazebo>
@@ -66,3 +66,10 @@
     damping="${damping}" friction="${friction}"
   />
+  <!-- ros_control-plugin -->
+  <gazebo>
+    <plugin name="gazebo_ros2_control" filename="libgazebo_ros2_control.so">
+      <parameters>$(find reachy_bringup)/config/reachy_controllers.yaml</parameters>
+      <robotNamespace>/reachy</robotNamespace>
+    </plugin>
+  </gazebo>
 </robot>
