Commit message: gazebo seems ok with cyclonedds

File: reachy_description/urdf/arm.urdf.xacro (robot description, xacro)
@@ -244,4 +244,22 @@
       <dynamics damping="${damping}" friction="${friction}"/>
   </joint>
+  <xacro:if value="$(arg use_gazebo)">
+    <gazebo reference="${prefix}_gripper">
+      <provideFeedback>true</provideFeedback>
+    </gazebo>
+    <gazebo>
+      <plugin name="gazebo_ros_ft" filename="libgazebo_ros_ft_sensor.so">
+        <ros>
+          <!-- Add namespace and remap the default topic -->
+          <namespace>/${prefix}_force_sensor</namespace>
+          <argument>wrench:=${prefix}_gripper_ft_sensor</argument>
+        </ros>
+        <joint_name>${prefix}_gripper</joint_name>
+        <update_rate>200</update_rate>
+        <update_rate>1</update_rate>
+        <gaussian_noise>0.01</gaussian_noise>
+      </plugin>
+    </gazebo>
+  </xacro:if>
   <xacro:arm_control
     name="${prefix}"

File: reachy_description/urdf/head.urdf.xacro (robot description, xacro)
@@ -1,202 +1,438 @@
 <?xml version="1.0"?>
 <robot xmlns:xacro="http://www.ros.org/wiki/xacro">
-<xacro:macro name="head" params="parent damping friction">
-  <xacro:include filename="$(find reachy_description)/ros2_control/head.ros2_control.xacro"/>
-  <joint name="neck_roll" type="revolute">
+  <xacro:arg name="depth_camera" default="true"/>
+  <xacro:property name="camera_link" value="0.05" /> <!-- Size of square 'camera' box -->
+  <xacro:property name="camera_convergence" value="0.0" /> <!-- convergence angle (rad) of the cameras. 0=parallel-->
+  <xacro:macro name="head" params="parent damping friction">
+    <xacro:include filename="$(find reachy_description)/ros2_control/head.ros2_control.xacro"/>
+    <joint name="neck_roll" type="revolute">
       <origin xyz="0.015 0.0 0.095" rpy="0 0.174 0" />
       <parent link="${parent}"/>
       <child link="head_x"/>
       <axis xyz="1 0 0"/>
-    <limit lower="-0.8" upper="0.8" effort="10." velocity="0.0"/>
-    <dynamics damping="${damping}" friction="${friction}"/>
-  </joint>
-  <link name="head_x">
-    <inertial>
-          <origin xyz="0.0 0.0 0.0" rpy="0.0 0.0 0.0"/>
-          <mass value="0.001"/>
-          <inertia ixx="1.0e-6" ixy="1.0e-8" ixz="1.0e-8" iyy="1.0e-6" iyz="1.0e-8" izz="1.0e-6"/>
-    </inertial>
-    </link>
-  <joint name="neck_pitch" type="revolute">
+      <limit lower="-0.8" upper="0.8" effort="10." velocity="0.0"/>
+      <dynamics damping="${damping}" friction="${friction}"/>
+    </joint>
+    <link name="head_x">
+      <inertial>
+        <origin xyz="0.0 0.0 0.0" rpy="0.0 0.0 0.0"/>
+        <mass value="0.001"/>
+        <inertia ixx="1.0e-6" ixy="1.0e-8" ixz="1.0e-8" iyy="1.0e-6" iyz="1.0e-8" izz="1.0e-6"/>
+      </inertial>
+    </link>
+    <joint name="neck_pitch" type="revolute">
       <origin xyz="0 0 0" rpy="0.0 0.0 0.0"/>
       <parent link="head_x"/>
       <child link="head_y"/>
       <axis xyz="0 1 0"/>
-    <limit lower="-0.8" upper="1.13" effort="10." velocity="0.0"/>
-    <dynamics damping="${damping}" friction="${friction}"/>
-  </joint>
-  <link name="head_y" >
-    <inertial>
-          <origin xyz="0.0 0.0 0.0" rpy="0.0 0.0 0.0"/>
-          <mass value="0.001"/>
-          <inertia ixx="1.0e-6" ixy="1.0e-8" ixz="1.0e-8" iyy="1.0e-6" iyz="1.0e-8" izz="1.0e-6"/>
-    </inertial>
-    </link>
-  <joint name="neck_yaw" type="revolute">
+      <limit lower="-0.8" upper="1.13" effort="10." velocity="0.0"/>
+      <dynamics damping="${damping}" friction="${friction}"/>
+    </joint>
+    <link name="head_y" >
+      <inertial>
+        <origin xyz="0.0 0.0 0.0" rpy="0.0 0.0 0.0"/>
+        <mass value="0.001"/>
+        <inertia ixx="1.0e-6" ixy="1.0e-8" ixz="1.0e-8" iyy="1.0e-6" iyz="1.0e-8" izz="1.0e-6"/>
+      </inertial>
+    </link>
+    <joint name="neck_yaw" type="revolute">
       <origin xyz="0 0 0" rpy="0.0 0.0 0.0"/>
       <parent link="head_y"/>
       <child link="head_z"/>
       <axis xyz="0 0 1"/>
-    <limit lower="-2.79" upper="2.79" effort="10." velocity="0.0"/>
-    <dynamics damping="${damping}" friction="${friction}"/>
-  </joint>
-  <link name="head_z">
-    <inertial>
-          <origin xyz="0.0 0.0 0.0" rpy="0.0 0.0 0.0"/>
-          <mass value="0.001"/>
-          <inertia ixx="1.0e-6" ixy="1.0e-8" ixz="1.0e-8" iyy="1.0e-6" iyz="1.0e-8" izz="1.0e-6"/>
-    </inertial>
-  </link>
-  <joint name="neck_fixed" type="fixed">
+      <limit lower="-2.79" upper="2.79" effort="10." velocity="0.0"/>
+      <dynamics damping="${damping}" friction="${friction}"/>
+    </joint>
+    <link name="head_z">
+      <inertial>
+        <origin xyz="0.0 0.0 0.0" rpy="0.0 0.0 0.0"/>
+        <mass value="0.001"/>
+        <inertia ixx="1.0e-6" ixy="1.0e-8" ixz="1.0e-8" iyy="1.0e-6" iyz="1.0e-8" izz="1.0e-6"/>
+      </inertial>
+    </link>
+    <joint name="neck_fixed" type="fixed">
       <origin xyz="0 0 0" rpy="0.0 0.0 0.0"/>
       <parent link="head_z" />
       <child link="head" />
-  </joint>
-  <!-- Fixed Orbita Arms Visuals -->
-  <joint name="neck_top" type="fixed">
+    </joint>
+    <!-- Fixed Orbita Arms Visuals -->
+    <joint name="neck_top" type="fixed">
       <origin xyz="0.0067 0.0 0.0478" rpy="0 0.174 0"/>
       <parent link="${parent}"/>
       <child link="top_neck_arm"/>
-  </joint>
-  <link name="top_neck_arm">
-    <inertial>
-          <origin xyz="0.0 0.0 0.0" rpy="0.0 0.0 0.0"/>
-          <mass value="0.001"/>
-          <inertia ixx="1.0e-6" ixy="1.0e-8" ixz="1.0e-8" iyy="1.0e-6" iyz="1.0e-8" izz="1.0e-6"/>
-    </inertial>
-      <visual name="">
-          <origin xyz="0.0 0.0 0.0" rpy="0.0 0.0 0.5236"/>
-          <geometry>
-              <mesh filename="file://$(find reachy_description)/meshes/orbita_arm.dae"/>
-          </geometry>
-      </visual>
-      <collision>
-          <origin xyz="0.0 0.0 0.0" rpy="0.0 0.0 0.0"/>
-          <geometry>
-              <cylinder length="0.0" radius="0.0" />
-          </geometry>
-      </collision>
-  </link>
-  <joint name="neck_middle" type="fixed">
+    </joint>
+    <link name="top_neck_arm">
+      <inertial>
+        <origin xyz="0.0 0.0 0.0" rpy="0.0 0.0 0.0"/>
+        <mass value="0.001"/>
+        <inertia ixx="1.0e-6" ixy="1.0e-8" ixz="1.0e-8" iyy="1.0e-6" iyz="1.0e-8" izz="1.0e-6"/>
+      </inertial>
+      <visual name="">
+        <origin xyz="0.0 0.0 0.0" rpy="0.0 0.0 0.5236"/>
+        <geometry>
+          <mesh filename="file://$(find reachy_description)/meshes/orbita_arm.dae"/>
+        </geometry>
+      </visual>
+      <collision>
+        <origin xyz="0.0 0.0 0.0" rpy="0.0 0.0 0.0"/>
+        <geometry>
+          <cylinder length="0.0" radius="0.0" />
+        </geometry>
+      </collision>
+    </link>
+    <joint name="neck_middle" type="fixed">
       <origin xyz="0.0067 0.0 0.0478" rpy="0 0.174 0"/>
       <parent link="${parent}"/>
       <child link="middle_neck_arm"/>
-  </joint>
-  <link name="middle_neck_arm">
-    <inertial>
-          <origin xyz="0.0 0.0 0.0" rpy="0.0 0.0 0.0"/>
-          <mass value="0.001"/>
-          <inertia ixx="1.0e-6" ixy="1.0e-8" ixz="1.0e-8" iyy="1.0e-6" iyz="1.0e-8" izz="1.0e-6"/>
-    </inertial>
-      <visual name="">
-          <origin xyz="0.0 0.0 0.0" rpy="0.0 0.0 2.618"/>
-          <geometry>
-              <mesh filename="file://$(find reachy_description)/meshes/orbita_arm.dae"/>
-          </geometry>
-      </visual>
-      <collision>
-          <origin xyz="0.0 0.0 0.0" rpy="0.0 0.0 0.0"/>
-          <geometry>
-              <cylinder length="0.0" radius="0.0" />
-          </geometry>
-      </collision>
-  </link>
-  <joint name="neck_bottom" type="fixed">
+    </joint>
+    <link name="middle_neck_arm">
+      <inertial>
+        <origin xyz="0.0 0.0 0.0" rpy="0.0 0.0 0.0"/>
+        <mass value="0.001"/>
+        <inertia ixx="1.0e-6" ixy="1.0e-8" ixz="1.0e-8" iyy="1.0e-6" iyz="1.0e-8" izz="1.0e-6"/>
+      </inertial>
+      <visual name="">
+        <origin xyz="0.0 0.0 0.0" rpy="0.0 0.0 2.618"/>
+        <geometry>
+          <mesh filename="file://$(find reachy_description)/meshes/orbita_arm.dae"/>
+        </geometry>
+      </visual>
+      <collision>
+        <origin xyz="0.0 0.0 0.0" rpy="0.0 0.0 0.0"/>
+        <geometry>
+          <cylinder length="0.0" radius="0.0" />
+        </geometry>
+      </collision>
+    </link>
+    <joint name="neck_bottom" type="fixed">
       <origin xyz="0.0067 0.0 0.0478" rpy="0 0.174 0"/>
       <parent link="${parent}"/>
       <child link="bottom_neck_arm"/>
-  </joint>
-  <link name="bottom_neck_arm">
-    <inertial>
-          <origin xyz="0.0 0.0 0.0" rpy="0.0 0.0 0.0"/>
-          <mass value="0.001"/>
-          <inertia ixx="1.0e-6" ixy="1.0e-8" ixz="1.0e-8" iyy="1.0e-6" iyz="1.0e-8" izz="1.0e-6"/>
-    </inertial>
-      <visual name="">
-          <origin xyz="0.0 0.0 0.0" rpy="0.0 0.0 -1.57"/>
-          <geometry>
-              <mesh filename="file://$(find reachy_description)/meshes/orbita_arm.dae"/>
-          </geometry>
-      </visual>
-      <collision>
-          <origin xyz="0.0 0.0 0.0" rpy="0.0 0.0 0.0"/>
-          <geometry>
-              <cylinder length="0.0" radius="0.0" />
-          </geometry>
-      </collision>
-  </link>
-  <!-- Head Links -->
-  <link name="head">
-      <inertial>
-          <origin xyz="-0.009 -0.002 0.059" rpy="0.0 0.0 0.0"/>
-          <mass value="0.237"/>
-          <inertia ixx="1.676e-3" ixy="3.068e-6" ixz="1.2449e-4" iyy="1.368e-3" iyz="3.360e-5" izz="8.425e-4"/>
-      </inertial>
-      <visual name="">
-          <origin xyz="0.0 0.0 0.0" rpy="0.0 0.0 0.0"/>
-          <geometry>
-              <mesh filename="file://$(find reachy_description)/meshes/head.dae"/>
-          </geometry>
-      </visual>
-      <collision>
-          <origin xyz="-0.009 -0.002 0.059" rpy="1.57 0.0 0.0"/>
-          <geometry>
-              <cylinder length="0.15" radius="0.06" />
-          </geometry>
-      </collision>
-  </link>
-  <link name="l_antenna_link">
-      <inertial>
-          <origin xyz="-0.001 0.0 0.008" rpy="0.0 0.0 0.0"/>
-          <mass value="0.004"/>
-          <inertia ixx="1.794e-7" ixy="-1.240e-5" ixz="1.91701e-8" iyy="1.5e-7" iyz="3.169e-6" izz="1.933e-7"/>
-      </inertial>
-      <visual name="">
-          <origin xyz="0.0 0.0 0.0" rpy="0.0 0.0 0.0"/>
-          <geometry>
-              <mesh filename="file://$(find reachy_description)/meshes/antenna.dae"/>
-          </geometry>
-      </visual>
-      <collision>
-          <origin xyz="0.1 0.0 0.1" rpy="0.0 0 0.0"/>
-          <geometry>
-              <cylinder length="0.0" radius="0.0" />
-          </geometry>
-      </collision>
-  </link>
-  <joint name="l_antenna" type="revolute">
+    </joint>
+    <link name="bottom_neck_arm">
+      <inertial>
+        <origin xyz="0.0 0.0 0.0" rpy="0.0 0.0 0.0"/>
+        <mass value="0.001"/>
+        <inertia ixx="1.0e-6" ixy="1.0e-8" ixz="1.0e-8" iyy="1.0e-6" iyz="1.0e-8" izz="1.0e-6"/>
+      </inertial>
+      <visual name="">
+        <origin xyz="0.0 0.0 0.0" rpy="0.0 0.0 -1.57"/>
+        <geometry>
+          <mesh filename="file://$(find reachy_description)/meshes/orbita_arm.dae"/>
+        </geometry>
+      </visual>
+      <collision>
+        <origin xyz="0.0 0.0 0.0" rpy="0.0 0.0 0.0"/>
+        <geometry>
+          <cylinder length="0.0" radius="0.0" />
+        </geometry>
+      </collision>
+    </link>
+    <!-- Head Links -->
+    <link name="head">
+      <inertial>
+        <origin xyz="-0.009 -0.002 0.059" rpy="0.0 0.0 0.0"/>
+        <mass value="0.237"/>
+        <inertia ixx="1.676e-3" ixy="3.068e-6" ixz="1.2449e-4" iyy="1.368e-3" iyz="3.360e-5" izz="8.425e-4"/>
+      </inertial>
+      <visual name="">
+        <origin xyz="0.0 0.0 0.0" rpy="0.0 0.0 0.0"/>
+        <geometry>
+          <mesh filename="file://$(find reachy_description)/meshes/head.dae"/>
+        </geometry>
+      </visual>
+      <collision>
+        <origin xyz="-0.009 -0.002 0.059" rpy="1.57 0.0 0.0"/>
+        <geometry>
+          <cylinder length="0.15" radius="0.06" />
+        </geometry>
+      </collision>
+    </link>
+    <link name="l_antenna_link">
+      <inertial>
+        <origin xyz="-0.001 0.0 0.008" rpy="0.0 0.0 0.0"/>
+        <mass value="0.004"/>
+        <inertia ixx="1.794e-7" ixy="-1.240e-5" ixz="1.91701e-8" iyy="1.5e-7" iyz="3.169e-6" izz="1.933e-7"/>
+      </inertial>
+      <visual name="">
+        <origin xyz="0.0 0.0 0.0" rpy="0.0 0.0 0.0"/>
+        <geometry>
+          <mesh filename="file://$(find reachy_description)/meshes/antenna.dae"/>
+        </geometry>
+      </visual>
+      <collision>
+        <origin xyz="0.1 0.0 0.1" rpy="0.0 0 0.0"/>
+        <geometry>
+          <cylinder length="0.0" radius="0.0" />
+        </geometry>
+      </collision>
+    </link>
+    <joint name="l_antenna" type="revolute">
       <origin xyz="-0.052 0.057 0.086" rpy="0.166 -1.054 -1.11"/>
       <parent link="head"/>
       <child link="l_antenna_link"/>
       <axis xyz="0 0 1"/>
-    <limit lower="-2.618" upper="2.618" effort="10." velocity="0.0"/>
-  </joint>
-  <link name="r_antenna_link">
-      <inertial>
-          <origin xyz="-0.001 0.0 0.008" rpy="0.0 0.0 0.0"/>
-          <mass value="0.004"/>
-          <inertia ixx="1.794e-7" ixy="-1.240e-5" ixz="1.91701e-8" iyy="1.5e-7" iyz="3.169e-6" izz="1.933e-7"/>
-      </inertial>
-      <visual name="">
-          <origin xyz="0.0 0.0 0.0" rpy="0.0 0.0 0.0"/>
-          <geometry>
-              <mesh filename="file://$(find reachy_description)/meshes/antenna.dae"/>
-          </geometry>
-      </visual>
-      <collision>
-          <origin xyz="0.0 0.0 0.0" rpy="0.0 0.0 0.0"/>
-          <geometry>
-              <cylinder length="0.0" radius="0.0" />
-          </geometry>
-      </collision>
-  </link>
-  <joint name="r_antenna" type="revolute">
+      <limit lower="-2.618" upper="2.618" effort="10." velocity="0.0"/>
+    </joint>
+    <link name="r_antenna_link">
+      <inertial>
+        <origin xyz="-0.001 0.0 0.008" rpy="0.0 0.0 0.0"/>
+        <mass value="0.004"/>
+        <inertia ixx="1.794e-7" ixy="-1.240e-5" ixz="1.91701e-8" iyy="1.5e-7" iyz="3.169e-6" izz="1.933e-7"/>
+      </inertial>
+      <visual name="">
+        <origin xyz="0.0 0.0 0.0" rpy="0.0 0.0 0.0"/>
+        <geometry>
+          <mesh filename="file://$(find reachy_description)/meshes/antenna.dae"/>
+        </geometry>
+      </visual>
+      <collision>
+        <origin xyz="0.0 0.0 0.0" rpy="0.0 0.0 0.0"/>
+        <geometry>
+          <cylinder length="0.0" radius="0.0" />
+        </geometry>
+      </collision>
+    </link>
+    <joint name="r_antenna" type="revolute">
       <origin xyz="-0.052 -0.057 0.086" rpy="-0.166 -1.054 1.11"/>
       <parent link="head"/>
       <child link="r_antenna_link"/>
       <axis xyz="0 0 1"/>
-    <limit lower="-2.618" upper="2.618" effort="10." velocity="0.0"/>
-  </joint>
-  <xacro:head_control/>
+      <limit lower="-2.618" upper="2.618" effort="10." velocity="0.0"/>
+    </joint>
+    <xacro:head_control/>
+    <!-- Cameras -->
+    <xacro:if value="$(arg use_gazebo)">
+      <joint name="left_cam_fixed" type="fixed">
+	<origin xyz="0.02 0.03625 0.06105" rpy="0.0 0.0  ${-camera_convergence/2.0}"/>
+	<parent link="head" />
+	<child link="left_camera" />
+      </joint>
+      <link name="left_camera" >
+	<!-- <collision> -->
+	<!--     <origin xyz="0 0 0" rpy="0 0 0"/> -->
+	<!--     <geometry> -->
+	<!--   <box size="${camera_link} ${camera_link} ${camera_link}"/> -->
+	<!--     </geometry> -->
+	<!--   </collision> -->
+	<!-- <visual> -->
+	<!--   <origin xyz="0 0 0" rpy="0 0 0"/> -->
+	<!--   <geometry> -->
+	<!-- <box size="${camera_link} ${camera_link} ${camera_link}"/> -->
+	<!--   </geometry> -->
+	<!--   <material name="red"/> -->
+	<!-- </visual> -->
+	<inertial>
+	  <mass value="1e-5" />
+	  <origin xyz="0 0 0" rpy="0 0 0"/>
+	  <inertia ixx="1e-6" ixy="0" ixz="0" iyy="1e-6" iyz="0" izz="1e-6" />
+	</inertial>
+      </link>
+      <link name="left_camera_optical">
+      </link>
+      <joint name="left_camera_optical_joint" type="fixed">
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
Commit message: cameras and force sensors should be SDK compatible

File: reachy_description/urdf/arm.urdf.xacro (robot description, xacro)
@@ -191,10 +191,17 @@
       </visual>
       <collision>
-          <origin xyz="0.0 0.02 -0.06" rpy="0.0 1.57 0.0"/>
-          <geometry>
-              <box size="0.1 0.012 0.035" />
-          </geometry>
-      </collision>
-  </link>
+          <origin xyz="0.0 0.0 0.0" rpy="0.0 1.57 0.0"/>
+          <geometry>
+              <mesh filename="file://$(find reachy_description)/meshes/${prefix}_gripper_thumb.dae"/>
+          </geometry>
+          <!-- <origin xyz="0.0 0.02 -0.06" rpy="0.0 1.57 0.0"/> -->
+          <!-- <geometry> -->
+          <!--     <box size="0.1 0.012 0.035" /> -->
+          <!-- </geometry> -->
+      </collision>
+  </link>
+  <gazebo reference="${prefix}_gripper_thumb">
+    <self_collide>1</self_collide>
+  </gazebo>
   <joint name="${prefix}_wrist_roll" type="revolute">
       <origin xyz="0 0 -0.0325" rpy="0.0 0.0 0.0"/>
@@ -218,10 +225,17 @@
       </visual>
       <collision>
-          <origin xyz="0.0 ${-0.01*reflect} -0.02" rpy="0.0 1.57 0.0"/>
-          <geometry>
-              <box size="0.1 0.012 0.035" />
-          </geometry>
-      </collision>
-  </link>
+          <origin xyz="0.0 0.0 0.0" rpy="0.0 1.57 0.0"/>
+          <geometry>
+              <mesh filename="file://$(find reachy_description)/meshes/${prefix}_gripper_finger.dae"/>
+          </geometry>
+          <!-- <origin xyz="0.0 ${-0.01*reflect} -0.02" rpy="0.0 1.57 0.0"/> -->
+          <!-- <geometry> -->
+          <!--     <box size="0.1 0.012 0.035" /> -->
+          <!-- </geometry> -->
+      </collision>
+  </link>
+  <gazebo reference="${prefix}_gripper_finger">
+    <self_collide>1</self_collide>
+  </gazebo>
   <link name="${prefix}_arm_tip">
     <inertial>
@@ -241,5 +255,10 @@
       <child link="${prefix}_gripper_finger"/>
       <axis xyz="1 0 0"/>
-      <limit lower="-1.2" upper="0.35" effort="10." velocity="0.0"/>
+      <xacro:if value="${side == 'right'}">
+        <limit lower="-1.2" upper="0.35" effort="10." velocity="0.0"/>
+      </xacro:if>
+      <xacro:if value="${side == 'left'}">
+        <limit lower="-0.35" upper="1.2" effort="10." velocity="0.0"/>
+      </xacro:if>
       <dynamics damping="${damping}" friction="${friction}"/>
   </joint>
@@ -262,4 +281,23 @@
     </gazebo>
   </xacro:if>
+  <!-- Doesn't work... -->
+  <!-- <xacro:if value="$(arg use_gazebo)"> -->
+  <!--   <gazebo reference="${prefix}_gripper_thumb"> -->
+  <!--     <provideFeedback>true</provideFeedback> -->
+  <!--   </gazebo> -->
+  <!--   <gazebo> -->
+  <!--     <plugin name="gazebo_ros_force_sensor" filename="libgazebo_ros_force.so"> -->
+  <!--       <ros> -->
+  <!--         <!-\- Add namespace and remap the default topic -\-> -->
+  <!--         <namespace>/${prefix}_force_sensor</namespace> -->
+  <!--       </ros> -->
+  <!--       <link_name>${prefix}_gripper_thumb</link_name> -->
+  <!--       <force_frame>world</force_frame> -->
+  <!--       <update_rate>200</update_rate> -->
+  <!--       <update_rate>1</update_rate> -->
+  <!--       <gaussian_noise>0.01</gaussian_noise> -->
+  <!--     </plugin> -->
+  <!--   </gazebo> -->
+  <!-- </xacro:if> -->
   <xacro:arm_control
     name="${prefix}"

File: reachy_description/urdf/head.urdf.xacro (robot description, xacro)
@@ -304,4 +304,10 @@
           <!-- Use camera, not camera_triggered -->
           <plugin name="left_camera_controller" filename="libgazebo_ros_camera.so">
+              <ros>
+                <namespace>/</namespace>
+                <remapping>image_raw:=image_raw</remapping>
+                <remapping>camera_info:=camera_info</remapping>
+              </ros>
+              <camera_name>left_image</camera_name>
             <!-- <ros> -->
             <!--   <namespace>custom_ns</namespace> -->
@@ -310,5 +316,5 @@
             <!-- </ros> -->
             <!-- Set camera name. If empty, defaults to sensor name (i.e. "sensor_name") -->
-            <camera_name>left_camera</camera_name>
+            <!-- <camera_name>left_camera</camera_name> -->
             <!-- Set TF frame name. If empty, defaults to link name (i.e. "link_name") -->
             <frame_name>left_camera_optical</frame_name>
@@ -347,4 +353,10 @@
           <!-- Use camera, not camera_triggered -->
           <plugin name="right_camera_controller" filename="libgazebo_ros_camera.so">
+              <ros>
+                <namespace>/</namespace>
+                <remapping>image_raw:=image_raw</remapping>
+                <remapping>camera_info:=camera_info</remapping>
+              </ros>
+              <camera_name>right_image</camera_name>
             <!-- <ros> -->
             <!--   <namespace>custom_ns</namespace> -->
@@ -353,5 +365,5 @@
             <!-- </ros> -->
             <!-- Set camera name. If empty, defaults to sensor name (i.e. "sensor_name") -->
-            <camera_name>right_camera</camera_name>
+            <!-- <camera_name>right_camera</camera_name> -->
             <!-- Set TF frame name. If empty, defaults to link name (i.e. "link_name") -->
             <frame_name>right_camera_optical</frame_name>

Commit message: Fix wrist roll limits

File: reachy_description/urdf/arm.urdf.xacro (robot description, xacro)
@@ -209,5 +209,10 @@
       <child link="${prefix}_gripper_thumb"/>
       <axis xyz="1 0 0"/>
-      <limit lower="-0.785" upper="0.785" effort="10." velocity="0.0"/>
+      <xacro:if value="${side == 'right'}">
+        <limit lower="-0.95" upper="0.61" effort="10." velocity="0.0"/>
+      </xacro:if>
+      <xacro:if value="${side == 'left'}">
+        <limit lower="-0.61" upper="0.95" effort="10." velocity="0.0"/>
+      </xacro:if>
       <dynamics damping="${damping}" friction="${friction}"/>
   </joint>
