Commit message: Added a second collision box to the finger to have a more realistic claw

File: reachy_description/urdf/arm.urdf.xacro (robot description, xacro)
@@ -227,5 +227,5 @@
                 <!-- <mesh filename="file://$(find reachy_description)/meshes/${prefix}_gripper_thumb.dae"/> -->
                 <!-- </geometry> -->
-                <origin xyz="0.0 ${0.02 *reflect} -0.06" rpy="0.0 1.57 0.0"/>
+                <origin xyz="0.0 ${0.02 *reflect} -0.06" rpy="-0.17 1.57 0.0"/>
                 <geometry>
                     <box size="0.1 0.012 0.035"/>
@@ -281,11 +281,32 @@
                 <!-- <mesh filename="file://$(find reachy_description)/meshes/${prefix}_gripper_finger.dae"/> -->
                 <!-- </geometry> -->
+                <origin xyz="0.0 ${-0.01*reflect} -0.02" rpy="0.17 1.57 0.0"/>
+                <geometry>
+                    <box size="0.05 0.012 0.035"/>
+                </geometry>
+            </collision>
+        </link>
+        <gazebo reference="${prefix}_gripper_finger">
+            <self_collide>1</self_collide>
+            <gravity>0</gravity>
+            <mu1>0.2</mu1>
+            <mu2>0.2</mu2>
+            <kp>2e+9</kp>
+            <kd>1.0</kd>
+        </gazebo>
+        <link name="${prefix}_gripper_finger2">
+            <inertial>
                 <origin xyz="0.0 ${-0.01*reflect} -0.02" rpy="0.0 1.57 0.0"/>
-                <geometry>
-                    <box size="0.1 0.012 0.035"/>
-                </geometry>
-            </collision>
-        </link>
-        <gazebo reference="${prefix}_gripper_finger">
+                <mass value="0.035"/>
+                <inertia ixx="1.062e-5" ixy="-6.559e-6" ixz="-3.952e-8" iyy="9.166e-5" iyz="5.276e-9" izz="8.704e-5"/>
+            </inertial>
+            <collision>
+                <origin xyz="0.0 ${-0.01*reflect} -0.02" rpy="0.17 1.57  -0.0"/>
+                <geometry>
+                    <box size="0.05 0.012 0.035"/>
+                </geometry>
+            </collision>
+        </link>
+        <gazebo reference="${prefix}_gripper_finger2">
             <self_collide>1</self_collide>
             <gravity>0</gravity>
@@ -307,6 +328,11 @@
             <child link="${prefix}_arm_tip"/>
         </joint>
+        <joint name="${prefix}_gripper_finger2" type="fixed">
+            <origin xyz="0.0 0.0 -0.05" rpy="${0.6*reflect} 0 0"/>
+            <parent link="${prefix}_gripper_finger"/>
+            <child link="${prefix}_gripper_finger2"/>
+        </joint>
         <joint name="${prefix}_gripper" type="revolute">
-            <origin xyz="0.0 ${-0.037*reflect} -0.03998" rpy="0.0 0.0 0.0"/>
+            <origin xyz="0.0 ${-0.037*reflect} -0.03998" rpy="-0.5 0.0 0.0"/>
             <parent link="${prefix}_gripper_thumb"/>
             <child link="${prefix}_gripper_finger"/>

Commit message: Bug #215: use package:// in xacro

File: reachy_description/urdf/arm.urdf.xacro (robot description, xacro)
@@ -21,5 +21,5 @@
                 <origin xyz="0.0 ${0.04*reflect} 0.0" rpy="${1.57*reflect} 1.57 0.0"/>
                 <geometry>
-                    <mesh filename="file://$(find reachy_description)/meshes/shoulder.dae"/>
+                    <mesh filename="package://reachy_description/meshes/shoulder.dae"/>
                 </geometry>
             </visual>
@@ -48,5 +48,5 @@
                 <origin xyz="0.0 0.0 0.0" rpy="0.0 0.0 0.0"/>
                 <geometry>
-                    <mesh filename="file://$(find reachy_description)/meshes/shoulder_x.dae"/>
+                    <mesh filename="package://reachy_description/meshes/shoulder_x.dae"/>
                 </geometry>
             </visual>
@@ -80,5 +80,5 @@
                 <origin xyz="0.0 0.0 -0.0526" rpy="0.0 0.0 0.0"/>
                 <geometry>
-                    <mesh filename="file://$(find reachy_description)/meshes/upper_arm.dae"/>
+                    <mesh filename="package://reachy_description/meshes/upper_arm.dae"/>
                 </geometry>
             </visual>
@@ -107,5 +107,5 @@
                 <origin xyz="0.0 0.0 0.0" rpy="0.0 0.0 0.0"/>
                 <geometry>
-                    <mesh filename="file://$(find reachy_description)/meshes/forearm.dae"/>
+                    <mesh filename="package://reachy_description/meshes/forearm.dae"/>
                 </geometry>
             </visual>
@@ -134,5 +134,5 @@
                 <origin xyz="0.0 0.0 -0.100" rpy="0.0 0.0 0.0"/>
                 <geometry>
-                    <mesh filename="file://$(find reachy_description)/meshes/wrist.dae"/>
+                    <mesh filename="package://reachy_description/meshes/wrist.dae"/>
                 </geometry>
             </visual>
@@ -171,5 +171,5 @@
                 <origin xyz="0.0 0.0 0.0" rpy="0.0 0.0 0.0"/>
                 <geometry>
-                    <mesh filename="file://$(find reachy_description)/meshes/wrist2hand.dae"/>
+                    <mesh filename="package://reachy_description/meshes/wrist2hand.dae"/>
                 </geometry>
             </visual>
@@ -216,5 +216,5 @@
                 <origin xyz="0.0 0.0 0.0" rpy="0.0 1.57 0.0"/>
                 <geometry>
-                    <mesh filename="file://$(find reachy_description)/meshes/${prefix}_gripper_thumb.dae"/>
+                    <mesh filename="package://reachy_description/meshes/${prefix}_gripper_thumb.dae"/>
                 </geometry>
             </visual>
@@ -222,5 +222,5 @@
                 <!-- <origin xyz="0.0 0.0 0.0" rpy="0.0 1.57 0.0"/> -->
                 <!-- <geometry> -->
-                <!-- <mesh filename="file://$(find reachy_description)/meshes/${prefix}_gripper_thumb.dae"/> -->
+                <!-- <mesh filename="package://reachy_description/meshes/${prefix}_gripper_thumb.dae"/> -->
                 <!-- </geometry> -->
                 <origin xyz="0.0 ${0.02 *reflect} -0.06" rpy="-0.17 1.57 0.0"/>
@@ -272,5 +272,5 @@
                 <origin xyz="0.0 0.0 0.0" rpy="0.0 1.57 0.0"/>
                 <geometry>
-                    <mesh filename="file://$(find reachy_description)/meshes/${prefix}_gripper_finger.dae"/>
+                    <mesh filename="package://reachy_description/meshes/${prefix}_gripper_finger.dae"/>
                 </geometry>
             </visual>
@@ -278,5 +278,5 @@
                 <!-- <origin xyz="0.0 0.0 0.0" rpy="0.0 1.57 0.0"/> -->
                 <!-- <geometry> -->
-                <!-- <mesh filename="file://$(find reachy_description)/meshes/${prefix}_gripper_finger.dae"/> -->
+                <!-- <mesh filename="package://reachy_description/meshes/${prefix}_gripper_finger.dae"/> -->
                 <!-- </geometry> -->
                 <origin xyz="0.0 ${-0.01*reflect} -0.02" rpy="0.17 1.57 0.0"/>

File: reachy_description/urdf/head.urdf.xacro (robot description, xacro)
@@ -71,5 +71,5 @@
         <origin xyz="0.0 0.0 0.0" rpy="0.0 0.0 0.5236"/>
         <geometry>
-          <mesh filename="file://$(find reachy_description)/meshes/orbita_arm.dae"/>
+          <mesh filename="package://reachy_description/meshes/orbita_arm.dae"/>
         </geometry>
       </visual>
@@ -95,5 +95,5 @@
         <origin xyz="0.0 0.0 0.0" rpy="0.0 0.0 2.618"/>
         <geometry>
-          <mesh filename="file://$(find reachy_description)/meshes/orbita_arm.dae"/>
+          <mesh filename="package://reachy_description/meshes/orbita_arm.dae"/>
         </geometry>
       </visual>
@@ -119,5 +119,5 @@
         <origin xyz="0.0 0.0 0.0" rpy="0.0 0.0 -1.57"/>
         <geometry>
-          <mesh filename="file://$(find reachy_description)/meshes/orbita_arm.dae"/>
+          <mesh filename="package://reachy_description/meshes/orbita_arm.dae"/>
         </geometry>
       </visual>
@@ -139,5 +139,5 @@
         <origin xyz="0.0 0.0 0.0" rpy="0.0 0.0 0.0"/>
         <geometry>
-          <mesh filename="file://$(find reachy_description)/meshes/head.dae"/>
+          <mesh filename="package://reachy_description/meshes/head.dae"/>
         </geometry>
       </visual>
@@ -168,5 +168,5 @@
         <origin xyz="0.0 0.0 0.0" rpy="0.0 0.0 0.0"/>
         <geometry>
-          <mesh filename="file://$(find reachy_description)/meshes/antenna.dae"/>
+          <mesh filename="package://reachy_description/meshes/antenna.dae"/>
         </geometry>
       </visual>
@@ -194,5 +194,5 @@
         <origin xyz="0.0 0.0 0.0" rpy="0.0 0.0 0.0"/>
         <geometry>
-          <mesh filename="file://$(find reachy_description)/meshes/antenna.dae"/>
+          <mesh filename="package://reachy_description/meshes/antenna.dae"/>
         </geometry>
       </visual>

File: reachy_description/urdf/meshed_arm.urdf.xacro (robot description, xacro)
@@ -20,5 +20,5 @@
           <origin xyz="0.0 ${0.04*reflect} 0.0" rpy="${1.57*reflect} 1.57 0.0"/>
           <geometry>
-              <mesh filename="file://$(find reachy_description)/meshes/shoulder.dae"/>
+              <mesh filename="package://reachy_description/meshes/shoulder.dae"/>
           </geometry>
       </visual>
@@ -47,5 +47,5 @@
           <origin xyz="0.0 0.0 0.0" rpy="0.0 0.0 0.0"/>
           <geometry>
-              <mesh filename="file://$(find reachy_description)/meshes/shoulder_x.dae"/>
+              <mesh filename="package://reachy_description/meshes/shoulder_x.dae"/>
           </geometry>
       </visual>
@@ -79,5 +79,5 @@
           <origin xyz="0.0 0.0 -0.0526" rpy="0.0 0.0 0.0"/>
           <geometry>
-              <mesh filename="file://$(find reachy_description)/meshes/upper_arm.dae"/>
+              <mesh filename="package://reachy_description/meshes/upper_arm.dae"/>
           </geometry>
       </visual>
@@ -106,5 +106,5 @@
           <origin xyz="0.0 0.0 0.0" rpy="0.0 0.0 0.0"/>
           <geometry>
-              <mesh filename="file://$(find reachy_description)/meshes/forearm.dae"/>
+              <mesh filename="package://reachy_description/meshes/forearm.dae"/>
           </geometry>
       </visual>
@@ -133,5 +133,5 @@
           <origin xyz="0.0 0.0 -0.100" rpy="0.0 0.0 0.0"/>
           <geometry>
-              <mesh filename="file://$(find reachy_description)/meshes/wrist.dae"/>
+              <mesh filename="package://reachy_description/meshes/wrist.dae"/>
           </geometry>
       </visual>
@@ -160,5 +160,5 @@
           <origin xyz="0.0 0.0 0.0" rpy="0.0 0.0 0.0"/>
           <geometry>
-              <mesh filename="file://$(find reachy_description)/meshes/wrist2hand.dae"/>
+              <mesh filename="package://reachy_description/meshes/wrist2hand.dae"/>
           </geometry>
       </visual>
@@ -187,5 +187,5 @@
           <origin xyz="0.0 0.0 0.0" rpy="0.0 1.57 0.0"/>
           <geometry>
-              <mesh filename="file://$(find reachy_description)/meshes/${prefix}_gripper_thumb.dae"/>
+              <mesh filename="package://reachy_description/meshes/${prefix}_gripper_thumb.dae"/>
           </geometry>
       </visual>
@@ -193,5 +193,5 @@
           <origin xyz="0.0 0.0 0.0" rpy="0.0 1.57 0.0"/>
           <geometry>
-              <mesh filename="file://$(find reachy_description)/meshes/${prefix}_gripper_thumb.dae"/>
+              <mesh filename="package://reachy_description/meshes/${prefix}_gripper_thumb.dae"/>
           </geometry>
           <!-- <origin xyz="0.0 0.02 -0.06" rpy="0.0 1.57 0.0"/> -->
@@ -226,5 +226,5 @@
           <origin xyz="0.0 0.0 0.0" rpy="0.0 1.57 0.0"/>
           <geometry>
-              <mesh filename="file://$(find reachy_description)/meshes/${prefix}_gripper_finger.dae"/>
+              <mesh filename="package://reachy_description/meshes/${prefix}_gripper_finger.dae"/>
           </geometry>
       </visual>
@@ -232,5 +232,5 @@
           <origin xyz="0.0 0.0 0.0" rpy="0.0 1.57 0.0"/>
           <geometry>
-              <mesh filename="file://$(find reachy_description)/meshes/${prefix}_gripper_finger.dae"/>
+              <mesh filename="package://reachy_description/meshes/${prefix}_gripper_finger.dae"/>
           </geometry>
           <!-- <origin xyz="0.0 ${-0.01*reflect} -0.02" rpy="0.0 1.57 0.0"/> -->

File: reachy_description/urdf/reachy.urdf.xacro (robot description, xacro)
@@ -22,5 +22,5 @@
             <origin xyz="0.0 0.0 0.0" rpy="0.0 0.0 0.0"/>
             <geometry>
-                <mesh filename="file://$(find reachy_description)/meshes/torso.dae"/>
+                <mesh filename="package://reachy_description/meshes/torso.dae"/>
             </geometry>
         </visual>

Commit message: Angle limits proposal. Works well for top grasps. Weird diff on wrist motor but tested on the old black Reachy

File: reachy_description/urdf/arm.urdf.xacro (robot description, xacro)
@@ -95,5 +95,5 @@
             <child link="${prefix}_upper_arm"/>
             <axis xyz="0 0 1"/>
-            <limit lower="-1.57" upper="1.57" effort="10." velocity="0.0"/>
+            <limit lower="-1.57" upper="3.14" effort="10." velocity="0.0"/>
             <dynamics damping="${damping}" friction="${friction}"/>
         </joint>
@@ -247,8 +247,8 @@
             <axis xyz="1 0 0"/>
             <xacro:if value="${side == 'right'}">
-                <limit lower="-0.95" upper="0.61" effort="10." velocity="0.0"/>
+                <limit lower="-0.6" upper="1.24" effort="10." velocity="0.0"/>
             </xacro:if>
             <xacro:if value="${side == 'left'}">
-                <limit lower="-0.61" upper="0.95" effort="10." velocity="0.0"/>
+                <limit lower="-1.24" upper="0.6" effort="10." velocity="0.0"/>
             </xacro:if>
             <dynamics damping="${damping}" friction="${friction}"/>
