Commit message: Handle robot config in reachy.urdf.xacro.
Handle robot config (either full kit or starter kit left/right).

File: reachy_description/urdf/reachy.urdf.xacro (robot description, xacro)
@@ -3,4 +3,5 @@
   <xacro:arg name="use_fake_hardware" default="false"/>
   <xacro:arg name="use_gazebo" default="false"/>
+  <xacro:arg name="robot_config" default="full_kit"/>
   <xacro:include filename="$(find reachy_description)/urdf/arm.urdf.xacro"/>
   <xacro:include filename="$(find reachy_description)/urdf/head.urdf.xacro"/>
@@ -37,32 +38,54 @@
   <xacro:property name="damping" value="0.1"/>
   <xacro:property name="friction" value="0.1"/>
-  <!-- RIGHT ARM-->
-  <xacro:arm
-    prefix="r" parent="torso" side="right"
-    damping="${damping}" friction="${friction}"
-    serial_port="/dev/usb2ax_right_arm"
-    mx_ids="10, 11, 12, 13, 14, 15, 16, 17"
-    offsets="1.57, 1.57, 0.0, 0.0, 0.0, 0.0, 0.0, 0.0"
-    is_direct="0.0, 0.0, 0.0, 0.0, 0.0, 0.0, 0.0, 1.0"
-    reductions="1.0, 1.0, 1.0, 1.0, 1.0, 1.0, 1.0, -2.0"
-    force_sensor_id="40"
-    fan_id="41"
-  />
-  <!-- LEFT ARM-->
-  <xacro:arm
-    prefix="l" parent="torso" side="left"
-    damping="${damping}" friction="${friction}"
-    serial_port="/dev/usb2ax_left_arm"
-    mx_ids="20, 21, 22, 23, 24, 25, 26, 27"
-    offsets="1.57, -1.57, 0.0, 0.0, 0.0, 0.0, 0.0, 0.0"
-    is_direct="1.0, 0.0, 0.0, 0.0, 0.0, 0.0, 0.0, 1.0"
-    reductions="1.0, 1.0, 1.0, 1.0, 1.0, 1.0, 1.0, -2.0"
-    force_sensor_id="50"
-    fan_id="51"
-  />
-  <!-- HEAD-->
-  <xacro:head
-    parent="torso"
-    damping="${damping}" friction="${friction}"
-  />
+  <xacro:property name="robot_config" value="$(arg robot_config)"/>
+  <xacro:if value="${robot_config == 'full_kit'}">
+    <xacro:property name="use_right_arm" value="true"/>
+    <xacro:property name="use_left_arm" value="true"/>
+    <xacro:property name="use_head" value="true"/>
+  </xacro:if>
+  <xacro:if value="${robot_config == 'starter_kit_left'}">
+    <xacro:property name="use_right_arm" value="false"/>
+    <xacro:property name="use_left_arm" value="true"/>
+    <xacro:property name="use_head" value="true"/>
+  </xacro:if>
+  <xacro:if value="${robot_config == 'starter_kit_right'}">
+    <xacro:property name="use_right_arm" value="true"/>
+    <xacro:property name="use_left_arm" value="false"/>
+    <xacro:property name="use_head" value="true"/>
+  </xacro:if>
+  <xacro:if value="${use_right_arm}">
+    <!-- RIGHT ARM-->
+    <xacro:arm
+      prefix="r" parent="torso" side="right"
+      damping="${damping}" friction="${friction}"
+      serial_port="/dev/usb2ax_right_arm"
+      mx_ids="10, 11, 12, 13, 14, 15, 16, 17"
+      offsets="1.57, 1.57, 0.0, 0.0, 0.0, 0.0, 0.0, 0.0"
+      is_direct="0.0, 0.0, 0.0, 0.0, 0.0, 0.0, 0.0, 1.0"
+      reductions="1.0, 1.0, 1.0, 1.0, 1.0, 1.0, 1.0, -2.0"
+      force_sensor_id="40"
+      fan_id="41"
+    />
+  </xacro:if>
+  <xacro:if value="${use_left_arm}">
+    <!-- LEFT ARM-->
+    <xacro:arm
+      prefix="l" parent="torso" side="left"
+      damping="${damping}" friction="${friction}"
+      serial_port="/dev/usb2ax_left_arm"
+      mx_ids="20, 21, 22, 23, 24, 25, 26, 27"
+      offsets="1.57, -1.57, 0.0, 0.0, 0.0, 0.0, 0.0, 0.0"
+      is_direct="1.0, 0.0, 0.0, 0.0, 0.0, 0.0, 0.0, 1.0"
+      reductions="1.0, 1.0, 1.0, 1.0, 1.0, 1.0, 1.0, -2.0"
+      force_sensor_id="50"
+      fan_id="51"
+    />
+  </xacro:if>
+  <xacro:if value="${use_head}">
+    <!-- HEAD-->
+    <xacro:head
+      parent="torso"
+      damping="${damping}" friction="${friction}"
+    />
+  </xacro:if>
 </robot>

Commit message: Slight improvement of reachy import mechanic Orbita zeroes are now loaded into urdf

File: reachy_description/urdf/reachy.urdf.xacro (robot description, xacro)
@@ -1,110 +1,111 @@
 <?xml version="1.0"?>
 <robot xmlns:xacro="http://www.ros.org/wiki/xacro" name="reachy_2023">
-  <xacro:arg name="use_fake_hardware" default="false"/>
-  <xacro:arg name="use_gazebo" default="false"/>
-  <xacro:arg name="robot_config" default="full_kit"/>
-  <xacro:include filename="$(find reachy_description)/urdf/arm.urdf.xacro"/>
-  <xacro:include filename="$(find reachy_description)/urdf/head.urdf.xacro"/>
-  <link name="world"/>
-  <joint name="world_joint" type="fixed">
-    <origin xyz="0 0 1.0" rpy="0 0 0"/>
-    <parent link="world"/>
-    <child link="torso"/>
-  </joint>
-  <link name="torso">
-      <inertial>
-          <origin xyz="0.0 0.019 -0.009" rpy="0.0 0.0 0.0"/>
-          <mass value="0.527"/>
-          <inertia ixx="2.89598e-3" ixy="-1.16791e-6" ixz="-8.28749e-6" iyy="4.491e-3" iyz="2.343e-4" izz="3.995e-3"/>
-      </inertial>
-      <visual name="">
-          <origin xyz="0.0 0.0 0.0" rpy="0.0 0.0 0.0"/>
-          <geometry>
-              <mesh filename="file://$(find reachy_description)/meshes/torso.dae"/>
-          </geometry>
-      </visual>
-      <collision>
-          <origin xyz="0 0 -0.1" rpy="0 0.05 0" />
-          <geometry>
-              <box size="0.11 0.2 0.32" />
-          </geometry>
-      </collision>
-  </link>
-  <gazebo reference="torso">
-    <material>Gazebo/White</material>
-    <static>true</static>
-  </gazebo>
-  <!--MODEL PARAMETERS-->
-  <xacro:property name="damping" value="0.1"/>
-  <xacro:property name="friction" value="0.1"/>
-  <xacro:property name="robot_config" value="$(arg robot_config)"/>
-  <xacro:if value="${robot_config == 'full_kit'}">
-    <xacro:property name="use_right_arm" value="true"/>
-    <xacro:property name="use_left_arm" value="true"/>
-    <xacro:property name="use_head" value="true"/>
-  </xacro:if>
-  <xacro:if value="${robot_config == 'starter_kit_left'}">
-    <xacro:property name="use_right_arm" value="false"/>
-    <xacro:property name="use_left_arm" value="true"/>
-    <xacro:property name="use_head" value="true"/>
-  </xacro:if>
-  <xacro:if value="${robot_config == 'starter_kit_right'}">
-    <xacro:property name="use_right_arm" value="true"/>
-    <xacro:property name="use_left_arm" value="false"/>
-    <xacro:property name="use_head" value="true"/>
-  </xacro:if>
-  <xacro:if value="${use_right_arm}">
-    <!-- RIGHT ARM-->
-    <xacro:arm
-      prefix="r" parent="torso" side="right"
-      damping="${damping}" friction="${friction}"
-      serial_port="/dev/usb2ax_right_arm"
-      mx_ids="10, 11, 12, 13, 14, 15, 16, 17"
-      offsets="1.57, 1.57, 0.0, 0.0, 0.0, 0.0, 0.0, 0.0"
-      is_direct="0.0, 0.0, 0.0, 0.0, 0.0, 0.0, 0.0, 1.0"
-      reductions="1.0, 1.0, 1.0, 1.0, 1.0, 1.0, 1.0, -2.0"
-      force_sensor_id="40"
-      fan_id="41"
-    />
-  </xacro:if>
-  <xacro:if value="${use_left_arm}">
-    <!-- LEFT ARM-->
-    <xacro:arm
-      prefix="l" parent="torso" side="left"
-      damping="${damping}" friction="${friction}"
-      serial_port="/dev/usb2ax_left_arm"
-      mx_ids="20, 21, 22, 23, 24, 25, 26, 27"
-      offsets="1.57, -1.57, 0.0, 0.0, 0.0, 0.0, 0.0, 0.0"
-      is_direct="1.0, 0.0, 0.0, 0.0, 0.0, 0.0, 0.0, 1.0"
-      reductions="1.0, 1.0, 1.0, 1.0, 1.0, 1.0, 1.0, -2.0"
-      force_sensor_id="50"
-      fan_id="51"
-    />
-  </xacro:if>
-  <xacro:if value="${use_head}">
-    <!-- HEAD-->
-    <xacro:head
-      parent="torso"
-      damping="${damping}" friction="${friction}"
-      neck_orbita_serial_port="/dev/orbita_neck"
-      neck_orbita_id="70"
-      neck_orbita_alpha="54.0"
-      neck_orbita_hardware_zero="0.4293648, 1.2923188, 0.018335864"
-      neck_orbita_reduction="4.26666667"
-      head_serial_port="/dev/usb2ax_head"
-      head_xl320_ids="30, 31"
-      head_xl320_offsets="0.0, 0.0"
-      head_xl320_is_direct="0.0, 0.0"
-      head_xl320_reductions="1.0, 1.0"
-      head_fan_id="60"
-    />
-  </xacro:if>
-  <xacro:if value="$(arg use_gazebo)">
-  <gazebo>
-    <plugin name="gazebo_ros2_control" filename="libgazebo_ros2_control.so">
-      <parameters>$(find reachy_bringup)/config/reachy_${robot_config}_controllers.yaml</parameters>
-      <robotNamespace>/reachy</robotNamespace>
-    </plugin>
-  </gazebo>
-  </xacro:if>
+    <xacro:arg name="use_fake_hardware" default="false"/>
+    <xacro:arg name="use_gazebo" default="false"/>
+    <xacro:arg name="robot_config" default="full_kit"/>
+    <xacro:arg name="orbita_hardware_zero" default="0.0, 0.0, 0.0"/>
+    <xacro:include filename="$(find reachy_description)/urdf/arm.urdf.xacro"/>
+    <xacro:include filename="$(find reachy_description)/urdf/head.urdf.xacro"/>
+    <link name="world"/>
+    <joint name="world_joint" type="fixed">
+        <origin xyz="0 0 1.0" rpy="0 0 0"/>
+        <parent link="world"/>
+        <child link="torso"/>
+    </joint>
+    <link name="torso">
+        <inertial>
+            <origin xyz="0.0 0.019 -0.009" rpy="0.0 0.0 0.0"/>
+            <mass value="0.527"/>
+            <inertia ixx="2.89598e-3" ixy="-1.16791e-6" ixz="-8.28749e-6" iyy="4.491e-3" iyz="2.343e-4" izz="3.995e-3"/>
+        </inertial>
+        <visual name="">
+            <origin xyz="0.0 0.0 0.0" rpy="0.0 0.0 0.0"/>
+            <geometry>
+                <mesh filename="file://$(find reachy_description)/meshes/torso.dae"/>
+            </geometry>
+        </visual>
+        <collision>
+            <origin xyz="0 0 -0.1" rpy="0 0.05 0"/>
+            <geometry>
+                <box size="0.11 0.2 0.32"/>
+            </geometry>
+        </collision>
+    </link>
+    <gazebo reference="torso">
+        <material>Gazebo/White</material>
+        <static>true</static>
+    </gazebo>
+    <!--MODEL PARAMETERS-->
+    <xacro:property name="damping" value="0.1"/>
+    <xacro:property name="friction" value="0.1"/>
+    <xacro:property name="robot_config" value="$(arg robot_config)"/>
+    <xacro:if value="${robot_config == 'full_kit'}">
+        <xacro:property name="use_right_arm" value="true"/>
+        <xacro:property name="use_left_arm" value="true"/>
+        <xacro:property name="use_head" value="true"/>
+    </xacro:if>
+    <xacro:if value="${robot_config == 'starter_kit_left'}">
+        <xacro:property name="use_right_arm" value="false"/>
+        <xacro:property name="use_left_arm" value="true"/>
+        <xacro:property name="use_head" value="true"/>
+    </xacro:if>
+    <xacro:if value="${robot_config == 'starter_kit_right'}">
+        <xacro:property name="use_right_arm" value="true"/>
+        <xacro:property name="use_left_arm" value="false"/>
+        <xacro:property name="use_head" value="true"/>
+    </xacro:if>
+    <xacro:if value="${use_right_arm}">
+        <!-- RIGHT ARM-->
+        <xacro:arm
+                prefix="r" parent="torso" side="right"
+                damping="${damping}" friction="${friction}"
+                serial_port="/dev/usb2ax_right_arm"
+                mx_ids="10, 11, 12, 13, 14, 15, 16, 17"
+                offsets="1.57, 1.57, 0.0, 0.0, 0.0, 0.0, 0.0, 0.0"
+                is_direct="0.0, 0.0, 0.0, 0.0, 0.0, 0.0, 0.0, 1.0"
+                reductions="1.0, 1.0, 1.0, 1.0, 1.0, 1.0, 1.0, -2.0"
+                force_sensor_id="40"
+                fan_id="41"
+        />
+    </xacro:if>
+    <xacro:if value="${use_left_arm}">
+        <!-- LEFT ARM-->
+        <xacro:arm
+                prefix="l" parent="torso" side="left"
+                damping="${damping}" friction="${friction}"
+                serial_port="/dev/usb2ax_left_arm"
+                mx_ids="20, 21, 22, 23, 24, 25, 26, 27"
+                offsets="1.57, -1.57, 0.0, 0.0, 0.0, 0.0, 0.0, 0.0"
+                is_direct="1.0, 0.0, 0.0, 0.0, 0.0, 0.0, 0.0, 1.0"
+                reductions="1.0, 1.0, 1.0, 1.0, 1.0, 1.0, 1.0, -2.0"
+                force_sensor_id="50"
+                fan_id="51"
+        />
+    </xacro:if>
+    <xacro:if value="${use_head}">
+        <!-- HEAD-->
+        <xacro:head
+                parent="torso"
+                damping="${damping}" friction="${friction}"
+                neck_orbita_serial_port="/dev/orbita_neck"
+                neck_orbita_id="70"
+                neck_orbita_alpha="54.0"
+                neck_orbita_hardware_zero="$(arg orbita_hardware_zero)"
+                neck_orbita_reduction="4.26666667"
+                head_serial_port="/dev/usb2ax_head"
+                head_xl320_ids="30, 31"
+                head_xl320_offsets="0.0, 0.0"
+                head_xl320_is_direct="0.0, 0.0"
+                head_xl320_reductions="1.0, 1.0"
+                head_fan_id="60"
+        />
+    </xacro:if>
+    <xacro:if value="$(arg use_gazebo)">
+        <gazebo>
+            <plugin name="gazebo_ros2_control" filename="libgazebo_ros2_control.so">
+                <parameters>$(find reachy_bringup)/config/reachy_${robot_config}_controllers.yaml</parameters>
+                <robotNamespace>/reachy</robotNamespace>
+            </plugin>
+        </gazebo>
+    </xacro:if>
 </robot>

Commit message: added headless mode for testing purpose has to be tested though...

File: reachy_description/urdf/reachy.urdf.xacro (robot description, xacro)
@@ -55,4 +55,9 @@
         <xacro:property name="use_head" value="true"/>
     </xacro:if>
+    <xacro:if value="${robot_config == 'headless'}">
+        <xacro:property name="use_right_arm" value="true"/>
+        <xacro:property name="use_left_arm" value="true"/>
+        <xacro:property name="use_head" value="false"/>
+    </xacro:if>
     <xacro:if value="${use_right_arm}">
         <!-- RIGHT ARM-->

Commit message: Add config for Reachy mini.

File: reachy_description/urdf/reachy.urdf.xacro (robot description, xacro)
@@ -60,4 +60,9 @@
         <xacro:property name="use_head" value="false"/>
     </xacro:if>
+    <xacro:if value="${robot_config == 'mini'}">
+        <xacro:property name="use_right_arm" value="false"/>
+        <xacro:property name="use_left_arm" value="false"/>
+        <xacro:property name="use_head" value="true"/>
+    </xacro:if>
     <xacro:if value="${use_right_arm}">
         <!-- RIGHT ARM-->

Commit message: merge : Add config for Reachy mini.

File: reachy_description/urdf/reachy.urdf.xacro (robot description, xacro)
@@ -77,4 +77,9 @@
         <xacro:property name="use_orbita" value="true"/>
     </xacro:if>
+    <xacro:if value="${robot_config == 'mini'}">
+        <xacro:property name="use_right_arm" value="false"/>
+        <xacro:property name="use_left_arm" value="false"/>
+        <xacro:property name="use_head" value="true"/>
+    </xacro:if>
     <xacro:if value="${use_right_arm}">
         <!-- RIGHT ARM-->

Commit message: Add custom config in reachy urdf.

File: reachy_description/urdf/reachy.urdf.xacro (robot description, xacro)
@@ -7,4 +7,5 @@
     <xacro:include filename="$(find reachy_description)/urdf/arm.urdf.xacro"/>
     <xacro:include filename="$(find reachy_description)/urdf/head.urdf.xacro"/>
+    <xacro:include filename="$(find reachy_description)/urdf/orbita.urdf.xacro"/>
     <link name="world"/>
     <joint name="world_joint" type="fixed">
@@ -44,4 +45,5 @@
         <xacro:property name="use_left_arm" value="true"/>
         <xacro:property name="use_head" value="true"/>
+        <xacro:property name="use_orbita" value="false"/>
     </xacro:if>
     <xacro:if value="${robot_config == 'starter_kit_left'}">
@@ -49,4 +51,5 @@
         <xacro:property name="use_left_arm" value="true"/>
         <xacro:property name="use_head" value="true"/>
+        <xacro:property name="use_orbita" value="false"/>
     </xacro:if>
     <xacro:if value="${robot_config == 'starter_kit_right'}">
@@ -54,4 +57,5 @@
         <xacro:property name="use_left_arm" value="false"/>
         <xacro:property name="use_head" value="true"/>
+        <xacro:property name="use_orbita" value="false"/>
     </xacro:if>
     <xacro:if value="${robot_config == 'headless'}">
@@ -59,4 +63,5 @@
         <xacro:property name="use_left_arm" value="true"/>
         <xacro:property name="use_head" value="false"/>
+        <xacro:property name="use_orbita" value="false"/>
     </xacro:if>
     <xacro:if value="${robot_config == 'mini'}">
@@ -64,4 +69,11 @@
         <xacro:property name="use_left_arm" value="false"/>
         <xacro:property name="use_head" value="true"/>
+        <xacro:property name="use_orbita" value="false"/>
+    </xacro:if>
+    <xacro:if value="${robot_config == 'starter_kit_right_no_head'}">
+        <xacro:property name="use_right_arm" value="true"/>
+        <xacro:property name="use_left_arm" value="false"/>
+        <xacro:property name="use_head" value="false"/>
+        <xacro:property name="use_orbita" value="true"/>
     </xacro:if>
     <xacro:if value="${use_right_arm}">
@@ -111,4 +123,16 @@
         />
     </xacro:if>
+    <xacro:if value="${use_orbita}">
+        <!-- NO HEAD CASE - ONLY ORBITA IS REQUIRED -->
+        <xacro:orbita
+                parent="torso"
+                damping="${damping}" friction="${friction}"
+                neck_orbita_serial_port="/dev/orbita_neck"
+                neck_orbita_id="70"
+                neck_orbita_alpha="0.9424777960769379"
+                neck_orbita_hardware_zero="$(arg orbita_hardware_zero)"
+                neck_orbita_reduction="4.26666667"
+        />
+    </xacro:if>
     <xacro:if value="$(arg use_gazebo)">
         <gazebo>

Commit message: Add right arm config.

File: reachy_description/urdf/reachy.urdf.xacro (robot description, xacro)
@@ -77,4 +77,10 @@
         <xacro:property name="use_orbita" value="true"/>
     </xacro:if>
+    <xacro:if value="${robot_config == 'right_arm'}">
+        <xacro:property name="use_right_arm" value="true"/>
+        <xacro:property name="use_left_arm" value="false"/>
+        <xacro:property name="use_head" value="false"/>
+        <xacro:property name="use_orbita" value="false"/>
+    </xacro:if>
     <xacro:if value="${use_right_arm}">
         <!-- RIGHT ARM-->

Commit message: Release 0.1.0 (#205)
* Update libneck_hwi.a from 4aa0ed182da61eef8e583dd67da99882  reachy_controllers/reachy_2023_controllers_rs/neck_hwi/target/debug/libneck_hwi.a to c1f572f1e4387567bcefe379714b3d65  reachy_controllers/reachy_2023_controllers_rs/neck_hwi/target/debug/libneck_hwi.a

* hotfix bad commit

* Update build_orbita_lib.yml

* Update build_orbita_lib.yml

* Update build_orbita_lib.yml

* Update build_orbita_lib.yml

* Update libneck_hwi.a

orbita3d_model_rs : 6099f8f8168faf4487a1105917a14793b8370f45
orbita_serial_controller : 27c23389bc1859f88cd29796da832a5959985c5a
libneck_hwi.a  : b08a8d1b0b4f120dc6c3fce18ae950d3

* Update libneck_hwi.a

orbita3d_model_rs : 6099f8f8168faf4487a1105917a14793b8370f45
orbita_serial_controller : 4648acb3533c1b2107ca058da55cf5e25b159c56
libneck_hwi.a  : 01d554041695e358ed13ea93603237a6

* License (#155)

* Create LICENSE

* Update LICENSE

* Update setup.py and package.xml of each package.

* Store latest motor discovery in dedicated yaml file.

Used by the dashboard to display the missing motors without having to disable reachy_sdk_server service to perform another scan.

* Add boolean to disable or not reachy_sdk_server when doing reachy -discovery.

* Perform motor discovery before launch ROS nodes in main launch file.

* Workaround fix to be able to load a custom Gazebo world

* Reverting erroneous PR merge

* Use reachy_utils to get zuuu_version.

* Update discovery.py

* 186 errors in discovery looked up ids (#187)

* Update looked up ids.

* Scan both protocol on head.

* Add config for Reachy mini.

* Update discovery.py (#190)

* Change logic for node spawning in launch file.

* Don't crash if no sensors are detected (the case for a Reachy mini).

* Change checking.

* Typo in main launch file. (#192)

* Create orbita ros2 control and urdf files.

* Add custom config in reachy urdf.

* Update reachy launch and discovery files.

* Create reachy_starter_kit_right_no_head_controllers.yaml

* Manage the condition for nodes that should not be spawned in headless and starter kit right configurations. (#203)

* 199 trigger the fans automatically if the motors get too hot (#201)

* Create fans controller package.

* Add fans controller to main launch file.

* Add fan_trigger_temperature parameter with default value to reachy.yaml

---------

Co-authored-by: CI <robot.setup@pollen-robotics.com>
Co-authored-by: Clément Dussieux <clement.dussieux@pollen-robotics.com>
Co-authored-by: cdussieux <clementdussieux@hotmail.fr>
Co-authored-by: RemiFabre <remifabre1800@gmail.com>
Co-authored-by: Pierre Rouanet <pierre.rouanet@gmail.com>

File: reachy_description/urdf/reachy.urdf.xacro (robot description, xacro)
@@ -7,4 +7,5 @@
     <xacro:include filename="$(find reachy_description)/urdf/arm.urdf.xacro"/>
     <xacro:include filename="$(find reachy_description)/urdf/head.urdf.xacro"/>
+    <xacro:include filename="$(find reachy_description)/urdf/orbita.urdf.xacro"/>
     <link name="world"/>
     <joint name="world_joint" type="fixed">
@@ -44,4 +45,5 @@
         <xacro:property name="use_left_arm" value="true"/>
         <xacro:property name="use_head" value="true"/>
+        <xacro:property name="use_orbita" value="false"/>
     </xacro:if>
     <xacro:if value="${robot_config == 'starter_kit_left'}">
@@ -49,4 +51,5 @@
         <xacro:property name="use_left_arm" value="true"/>
         <xacro:property name="use_head" value="true"/>
+        <xacro:property name="use_orbita" value="false"/>
     </xacro:if>
     <xacro:if value="${robot_config == 'starter_kit_right'}">
@@ -54,4 +57,5 @@
         <xacro:property name="use_left_arm" value="false"/>
         <xacro:property name="use_head" value="true"/>
+        <xacro:property name="use_orbita" value="false"/>
     </xacro:if>
     <xacro:if value="${robot_config == 'headless'}">
@@ -59,4 +63,17 @@
         <xacro:property name="use_left_arm" value="true"/>
         <xacro:property name="use_head" value="false"/>
+        <xacro:property name="use_orbita" value="false"/>
+    </xacro:if>
+    <xacro:if value="${robot_config == 'mini'}">
+        <xacro:property name="use_right_arm" value="false"/>
+        <xacro:property name="use_left_arm" value="false"/>
+        <xacro:property name="use_head" value="true"/>
+        <xacro:property name="use_orbita" value="false"/>
+    </xacro:if>
+    <xacro:if value="${robot_config == 'starter_kit_right_no_head'}">
+        <xacro:property name="use_right_arm" value="true"/>
+        <xacro:property name="use_left_arm" value="false"/>
+        <xacro:property name="use_head" value="false"/>
+        <xacro:property name="use_orbita" value="true"/>
     </xacro:if>
     <xacro:if value="${use_right_arm}">
@@ -106,4 +123,16 @@
         />
     </xacro:if>
+    <xacro:if value="${use_orbita}">
+        <!-- NO HEAD CASE - ONLY ORBITA IS REQUIRED -->
+        <xacro:orbita
+                parent="torso"
+                damping="${damping}" friction="${friction}"
+                neck_orbita_serial_port="/dev/orbita_neck"
+                neck_orbita_id="70"
+                neck_orbita_alpha="0.9424777960769379"
+                neck_orbita_hardware_zero="$(arg orbita_hardware_zero)"
+                neck_orbita_reduction="4.26666667"
+        />
+    </xacro:if>
     <xacro:if value="$(arg use_gazebo)">
         <gazebo>
