Commit message: Remove incorrect adding.

File: reachy_description/urdf/reachy.urdf.xacro (robot description, xacro)
@@ -77,9 +77,4 @@
         <xacro:property name="use_orbita" value="true"/>
     </xacro:if>
-    <xacro:if value="${robot_config == 'mini'}">
-        <xacro:property name="use_right_arm" value="false"/>
-        <xacro:property name="use_left_arm" value="false"/>
-        <xacro:property name="use_head" value="true"/>
-    </xacro:if>
     <xacro:if value="${use_right_arm}">
         <!-- RIGHT ARM-->

Commit message: Add orbita config.

File: reachy_description/urdf/reachy.urdf.xacro (robot description, xacro)
@@ -77,4 +77,10 @@
         <xacro:property name="use_orbita" value="true"/>
     </xacro:if>
+    <xacro:if value="${robot_config == 'orbita'}">
+        <xacro:property name="use_right_arm" value="false"/>
+        <xacro:property name="use_left_arm" value="false"/>
+        <xacro:property name="use_head" value="false"/>
+        <xacro:property name="use_orbita" value="true"/>
+    </xacro:if>
     <xacro:if value="${use_right_arm}">
         <!-- RIGHT ARM-->
